File: KICAD/CPU_ESP/V0.1/CPU/Power.kicad_sch (KiCad schematic)
At the start: 7 parts, among them U2 LM1117DT-2.5

Commit message: Update
Parts:
- C301: renamed from 22µ301; footprint (none) -> Capacitor_Tantalum_SMD:CP_EIA-3216-10_Kemet-I
- C304: renamed from C6; footprint (none) -> Capacitor_Tantalum_SMD:CP_EIA-3528-21_Kemet-B
- renumbered C8 to C302, C7 to C303, D1 to D301, R2 to R301, U2 to U301
Changed lines of the file:
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@@
 		(dnp no)
 		(fields_autoplaced yes)
-		(property "Reference" "#PWR07"
+		(property "Reference" "#PWR0308"
 			(at 176.53 73.66 0)
 			(effects
@@
 			(project ""
 				(path "/a676c576-12a0-418f-9fc1-1ecc8cb5a083/dfa41f31-372e-4922-9bef-c0e343f2f76b"
-					(reference "#PWR07")
+					(reference "#PWR0308")
 					(unit 1)
 				)
@@
 		(dnp no)
 		(fields_autoplaced yes)
-		(property "Reference" "D1"
+		(property "Reference" "D301"
 			(at 106.68 77.7874 90)
 			(effects
@@
 			(project ""
 				(path "/a676c576-12a0-418f-9fc1-1ecc8cb5a083/dfa41f31-372e-4922-9bef-c0e343f2f76b"
-					(reference "D1")
+					(reference "D301")
 					(unit 1)
 				)
@@
 		(dnp no)
 		(fields_autoplaced yes)
-		(property "Reference" "U2"
+		(property "Reference" "U301"
 			(at 146.05 66.04 0)
 			(effects
@@
 			(project ""
 				(path "/a676c576-12a0-418f-9fc1-1ecc8cb5a083/dfa41f31-372e-4922-9bef-c0e343f2f76b"
-					(reference "U2")
+					(reference "U301")
 					(unit 1)
 				)
@@
 		(dnp no)
 		(fields_autoplaced yes)
-		(property "Reference" "C7"
+		(property "Reference" "C303"
 			(at 163.83 74.9362 0)
 			(effects
@@
 			(project ""
 				(path "/a676c576-12a0-418f-9fc1-1ecc8cb5a083/dfa41f31-372e-4922-9bef-c0e343f2f76b"
-					(reference "C7")
+					(reference "C303")
 					(unit 1)
 				)
@@
 		(dnp no)
 		(fields_autoplaced yes)
-		(property "Reference" "#PWR0301"
+		(property "Reference" "#PWR0303"
 			(at 115.57 87.63 0)
 			(effects
@@
 			(project ""
 				(path "/a676c576-12a0-418f-9fc1-1ecc8cb5a083/dfa41f31-372e-4922-9bef-c0e343f2f76b"
-					(reference "#PWR0301")
+					(reference "#PWR0303")
 					(unit 1)
 				)
@@
 		(dnp no)
 		(fields_autoplaced yes)
-		(property "Reference" "#PWR0304"
+		(property "Reference" "#PWR0306"
 			(at 161.29 87.63 0)
 			(effects
@@
 			(project ""
 				(path "/a676c576-12a0-418f-9fc1-1ecc8cb5a083/dfa41f31-372e-4922-9bef-c0e343f2f76b"
-					(reference "#PWR0304")
+					(reference "#PWR0306")
 					(unit 1)
 				)
@@
 		(dnp no)
 		(fields_autoplaced yes)
-		(property "Reference" "#PWR0305"
+		(property "Reference" "#PWR0307"
 			(at 171.45 87.63 0)
 			(effects
@@
 			(project ""
 				(path "/a676c576-12a0-418f-9fc1-1ecc8cb5a083/dfa41f31-372e-4922-9bef-c0e343f2f76b"
-					(reference "#PWR0305")
+					(reference "#PWR0307")
 					(unit 1)
 				)
@@
 		(dnp no)
 		(fields_autoplaced yes)
-		(property "Reference" "#PWR08"
+		(property "Reference" "#PWR0301"
 			(at 102.87 100.33 0)
 			(effects
@@
 			(project ""
 				(path "/a676c576-12a0-418f-9fc1-1ecc8cb5a083/dfa41f31-372e-4922-9bef-c0e343f2f76b"
-					(reference "#PWR08")
+					(reference "#PWR0301")
 					(unit 1)
 				)
@@
 		(dnp no)
 		(fields_autoplaced yes)
-		(property "Reference" "#PWR0302"
+		(property "Reference" "#PWR0304"
 			(at 124.46 87.63 0)
 			(effects
@@
 			(project ""
 				(path "/a676c576-12a0-418f-9fc1-1ecc8cb5a083/dfa41f31-372e-4922-9bef-c0e343f2f76b"
-					(reference "#PWR0302")
+					(reference "#PWR0304")
 					(unit 1)
 				)
@@
 		(dnp no)
 		(fields_autoplaced yes)
-		(property "Reference" "#PWR0303"
+		(property "Reference" "#PWR0305"
 			(at 146.05 88.9 0)
 			(effects
@@
 			(project ""
 				(path "/a676c576-12a0-418f-9fc1-1ecc8cb5a083/dfa41f31-372e-4922-9bef-c0e343f2f76b"
-					(reference "#PWR0303")
+					(reference "#PWR0305")
 					(unit 1)
 				)
@@
 		(dnp no)
 		(fields_autoplaced yes)
-		(property "Reference" "C6"
+		(property "Reference" "C304"
 			(at 173.99 74.3838 0)
 			(effects
@@
 			)
 		)
-		(property "Footprint" ""
+		(property "Footprint" "Capacitor_Tantalum_SMD:CP_EIA-3528-21_Kemet-B"
 			(at 171.45 76.2 0)
 			(effects
@@
 			)
 		)
+		(property "TITLE" ""
+			(at 171.45 76.2 0)
+			(effects
+				(font
+					(size 1.27 1.27)
+				)
+				(hide yes)
+			)
+		)
 		(pin "1"
 		)
@@
 			(project ""
 				(path "/a676c576-12a0-418f-9fc1-1ecc8cb5a083/dfa41f31-372e-4922-9bef-c0e343f2f76b"
-					(reference "C6")
+					(reference "C304")
 					(unit 1)
 				)
@@
 		(dnp no)
 		(fields_autoplaced yes)
-		(property "Reference" "C8"
+		(property "Reference" "C302"
 			(at 127 74.9362 0)
 			(effects
@@
 			(project ""
 				(path "/a676c576-12a0-418f-9fc1-1ecc8cb5a083/dfa41f31-372e-4922-9bef-c0e343f2f76b"
-					(reference "C8")
+					(reference "C302")
 					(unit 1)
 				)
@@
 		(dnp no)
 		(fields_autoplaced yes)
-		(property "Reference" "R2"
+		(property "Reference" "R301"
 			(at 105.41 86.3599 0)
 			(effects
@@
 			(project ""
 				(path "/a676c576-12a0-418f-9fc1-1ecc8cb5a083/dfa41f31-372e-4922-9bef-c0e343f2f76b"
-					(reference "R2")
+					(reference "R301")
 					(unit 1)
 				)
@@
 		(dnp no)
 		(fields_autoplaced yes)
-		(property "Reference" "#PWR06"
+		(property "Reference" "#PWR0302"
 			(at 110.49 74.93 0)
 			(effects
@@
 			(project ""
 				(path "/a676c576-12a0-418f-9fc1-1ecc8cb5a083/dfa41f31-372e-4922-9bef-c0e343f2f76b"
-					(reference "#PWR06")
+					(reference "#PWR0302")
 					(unit 1)
 				)
@@
 		(dnp no)
 		(fields_autoplaced yes)
-		(property "Reference" "22µ301"
+		(property "Reference" "C301"
 			(at 118.11 74.3838 0)
 			(effects
@@
 			)
 		)
-		(property "Footprint" ""
+		(property "Footprint" "Capacitor_Tantalum_SMD:CP_EIA-3216-10_Kemet-I"
 			(at 115.57 76.2 0)
 			(effects
@@
 			)
 		)
+		(property "TITLE" ""
+			(at 115.57 76.2 0)
+			(effects
+				(font
+					(size 1.27 1.27)
+				)
+				(hide yes)
+			)
+		)
 		(pin "2"
 		)
@@
 			(project ""
 				(path "/a676c576-12a0-418f-9fc1-1ecc8cb5a083/dfa41f31-372e-4922-9bef-c0e343f2f76b"
-					(reference "22µ301")
-					(unit 1)
-				)
+					(reference "C301")
+					(unit 1)
+				)

Commit message: update
Other:
- company: (none) -> CMOS-74A
- title: (none) -> POWER SUPPLY
Changed lines of the file:
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@@
 	(generator_version "9.0")
 	(paper "A4")
+	(title_block
+		(title "POWER SUPPLY")
+		(date "2025-09-17")
+		(rev "V1.0")
+		(company "CMOS-74A")
+	)
 	(text "800mA"
 		(exclude_from_sim no)
