File: KICAD/CPU_ESP/V0.1/CPU/cmos_bus.kicad_sch (KiCad schematic)
At the start: 2 parts, among them J501 Conn_02x20_Odd_Even, J502 Conn_02x20_Odd_Even

Commit message: Update
Connections:
- net RST renamed RESET
Changed lines of the file:
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@@
 		)
 	)
-	(hierarchical_label "RST"
+	(hierarchical_label "RESET"
 		(shape input)
 		(at 151.13 113.03 180)

Commit message: update
Other:
- company: (none) -> CMOS-74A
- title: (none) -> BUS CMOS
Changed lines of the file:
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@@
 	(generator_version "9.0")
 	(paper "A4")
+	(title_block
+		(title "BUS CMOS")
+		(date "2025-09-17")
+		(rev "V1.0")
+		(company "CMOS-74A")
+	)
 	(wire
 		(pts
