File: KICAD/CPU_ESP/V0.1/CPU/ESP32.kicad_sch (KiCad schematic)
At the start: 6 parts, among them U1 ESP32-WROOM-32

Commit message: Update
Parts:
- C401: renamed from C3; value C_Small -> 100n; footprint (none) -> Capacitor_SMD:C_0603_1608Metric
- C402: renamed from C2; value C_Polarized_Small -> 22µ/10V; footprint (none) -> Capacitor_Tantalum_SMD:CP_EIA-3216-10_Kemet-I
- C403: renamed from C1; value C_Small -> 100n; footprint (none) -> Capacitor_SMD:C_0603_1608Metric
- C404: renamed from C4; value C_Small -> 100n; footprint (none) -> Capacitor_SMD:C_0603_1608Metric
- R401: renamed from R1; value R -> 10k; footprint (none) -> Resistor_SMD:R_0603_1608Metric
- renumbered U1 to U401
Changed lines of the file:
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@@
 		(dnp no)
 		(fields_autoplaced yes)
-		(property "Reference" "#PWR05"
+		(property "Reference" "#PWR0401"
 			(at 91.44 43.18 0)
 			(effects
@@
 			(project ""
 				(path "/a676c576-12a0-418f-9fc1-1ecc8cb5a083/3fae016e-6e0f-4cd9-b4b1-dc965be68ffa"
-					(reference "#PWR05")
+					(reference "#PWR0401")
 					(unit 1)
 				)
@@
 		(dnp no)
 		(fields_autoplaced yes)
-		(property "Reference" "#PWR02"
+		(property "Reference" "#PWR0403"
 			(at 106.68 27.94 0)
 			(effects
@@
 			(project ""
 				(path "/a676c576-12a0-418f-9fc1-1ecc8cb5a083/3fae016e-6e0f-4cd9-b4b1-dc965be68ffa"
-					(reference "#PWR02")
+					(reference "#PWR0403")
 					(unit 1)
 				)
@@
 		(dnp no)
 		(fields_autoplaced yes)
-		(property "Reference" "C3"
+		(property "Reference" "C401"
 			(at 93.98 53.3462 0)
 			(effects
@@
 			)
 		)
-		(property "Value" "C_Small"
+		(property "Value" "100n"
 			(at 93.98 55.8862 0)
 			(effects
@@
 			)
 		)
-		(property "Footprint" ""
+		(property "Footprint" "Capacitor_SMD:C_0603_1608Metric"
 			(at 91.44 54.61 0)
 			(effects
@@
 			)
 		)
+		(property "TITLE" ""
+			(at 91.44 54.61 0)
+			(effects
+				(font
+					(size 1.27 1.27)
+				)
+				(hide yes)
+			)
+		)
 		(pin "1"
 		)
@@
 			(project ""
 				(path "/a676c576-12a0-418f-9fc1-1ecc8cb5a083/3fae016e-6e0f-4cd9-b4b1-dc965be68ffa"
-					(reference "C3")
+					(reference "C401")
 					(unit 1)
 				)
@@
 		(dnp no)
 		(fields_autoplaced yes)
-		(property "Reference" "C2"
+		(property "Reference" "C402"
 			(at 109.22 27.3938 0)
 			(effects
@@
 			)
 		)
-		(property "Value" "C_Polarized_Small"
+		(property "Value" "22µ/10V"
 			(at 109.22 29.9338 0)
 			(effects
@@
 			)
 		)
-		(property "Footprint" ""
+		(property "Footprint" "Capacitor_Tantalum_SMD:CP_EIA-3216-10_Kemet-I"
 			(at 106.68 29.21 0)
 			(effects
@@
 			)
 		)
+		(property "TITLE" ""
+			(at 106.68 29.21 0)
+			(effects
+				(font
+					(size 1.27 1.27)
+				)
+				(hide yes)
+			)
+		)
 		(pin "1"
 		)
@@
 			(project ""
 				(path "/a676c576-12a0-418f-9fc1-1ecc8cb5a083/3fae016e-6e0f-4cd9-b4b1-dc965be68ffa"
-					(reference "C2")
+					(reference "C402")
 					(unit 1)
 				)
@@
 		(dnp no)
 		(fields_autoplaced yes)
-		(property "Reference" "C4"
+		(property "Reference" "C404"
 			(at 191.77 52.0762 0)
 			(effects
@@
 			)
 		)
-		(property "Value" "C_Small"
+		(property "Value" "100n"
 			(at 191.77 54.6162 0)
 			(effects
@@
 			)
 		)
-		(property "Footprint" ""
+		(property "Footprint" "Capacitor_SMD:C_0603_1608Metric"
 			(at 189.23 53.34 0)
 			(effects
@@
 			)
 		)
+		(property "TITLE" ""
+			(at 189.23 53.34 0)
+			(effects
+				(font
+					(size 1.27 1.27)
+				)
+				(hide yes)
+			)
+		)
 		(pin "2"
 		)
@@
 			(project ""
 				(path "/a676c576-12a0-418f-9fc1-1ecc8cb5a083/3fae016e-6e0f-4cd9-b4b1-dc965be68ffa"
-					(reference "C4")
+					(reference "C404")
 					(unit 1)
 				)
@@
 		(dnp no)
 		(fields_autoplaced yes)
-		(property "Reference" "R1"
+		(property "Reference" "R401"
 			(at 93.98 43.1799 0)
 			(effects
@@
 			)
 		)
-		(property "Value" "R"
+		(property "Value" "10k"
 			(at 93.98 45.7199 0)
 			(effects
@@
 			)
 		)
-		(property "Footprint" ""
+		(property "Footprint" "Resistor_SMD:R_0603_1608Metric"
 			(at 93.218 44.45 90)
 			(effects
@@
 			)
 		)
+		(property "TITLE" ""
+			(at 91.44 44.45 0)
+			(effects
+				(font
+					(size 1.27 1.27)
+				)
+				(hide yes)
+			)
+		)
 		(pin "1"
 		)
@@
 			(project ""
 				(path "/a676c576-12a0-418f-9fc1-1ecc8cb5a083/3fae016e-6e0f-4cd9-b4b1-dc965be68ffa"
-					(reference "R1")
+					(reference "R401")
 					(unit 1)
 				)
@@
 		(dnp no)
 		(fields_autoplaced yes)
-		(property "Reference" "#PWR04"
+		(property "Reference" "#PWR0406"
 			(at 189.23 63.5 0)
 			(effects
@@
 			(project ""
 				(path "/a676c576-12a0-418f-9fc1-1ecc8cb5a083/3fae016e-6e0f-4cd9-b4b1-dc965be68ffa"
-					(reference "#PWR04")
+					(reference "#PWR0406")
 					(unit 1)
 				)
@@
 		(dnp no)
 		(fields_autoplaced yes)
-		(property "Reference" "#PWR0401"
+		(property "Reference" "#PWR0405"
 			(at 151.13 125.73 0)
 			(effects
@@
 			(project ""
 				(path "/a676c576-12a0-418f-9fc1-1ecc8cb5a083/3fae016e-6e0f-4cd9-b4b1-dc965be68ffa"
-					(reference "#PWR0401")
+					(reference "#PWR0405")
 					(unit 1)
 				)
@@
 		(dnp no)
 		(fields_autoplaced yes)
-		(property "Reference" "C1"
+		(property "Reference" "C403"
 			(at 121.92 27.9462 0)
 			(effects
@@
 			)
 		)
-		(property "Value" "C_Small"
+		(property "Value" "100n"
 			(at 121.92 30.4862 0)
 			(effects
@@
 			)
 		)
-		(property "Footprint" ""
+		(property "Footprint" "Capacitor_SMD:C_0603_1608Metric"
 			(at 119.38 29.21 0)
 			(effects
@@
 			)
 		)
+		(property "TITLE" ""
+			(at 119.38 29.21 0)
+			(effects
+				(font
+					(size 1.27 1.27)
+				)
+				(hide yes)
+			)
+		)
 		(pin "2"
 		)
@@
 			(project ""
 				(path "/a676c576-12a0-418f-9fc1-1ecc8cb5a083/3fae016e-6e0f-4cd9-b4b1-dc965be68ffa"
-					(reference "C1")
+					(reference "C403")
 					(unit 1)
 				)
@@
 		(dnp no)
 		(fields_autoplaced yes)
-		(property "Reference" "U1"
+		(property "Reference" "U401"
 			(at 153.2733 43.18 0)
 			(effects
@@
 			(project ""
 				(path "/a676c576-12a0-418f-9fc1-1ecc8cb5a083/3fae016e-6e0f-4cd9-b4b1-dc965be68ffa"
-					(reference "U1")
+					(reference "U401")
 					(unit 1)
 				)
@@
 		(dnp no)
 		(fields_autoplaced yes)
-		(property "Reference" "#PWR03"
+		(property "Reference" "#PWR0402"
 			(at 91.44 64.77 0)
 			(effects
@@
 			(project ""
 				(path "/a676c576-12a0-418f-9fc1-1ecc8cb5a083/3fae016e-6e0f-4cd9-b4b1-dc965be68ffa"
-					(reference "#PWR03")
+					(reference "#PWR0402")
 					(unit 1)
 				)
@@
 		(dnp no)
 		(fields_autoplaced yes)
-		(property "Reference" "#PWR01"
+		(property "Reference" "#PWR0404"
 			(at 106.68 40.64 0)
 			(effects
@@
 			(project ""
 				(path "/a676c576-12a0-418f-9fc1-1ecc8cb5a083/3fae016e-6e0f-4cd9-b4b1-dc965be68ffa"
-					(reference "#PWR01")
-					(unit 1)
-				)
+					(reference "#PWR0404")
+					(unit 1)
+				)

Commit message: Update
Connections:
- net SDA: now reaches U401.33 (IO21)
- net RX0: now reaches U401.34 (RXD0/IO3)
- net TX0: now reaches U401.35 (TXD0/IO1)
- net SCL: now reaches U401.36 (IO22)

Commit message: update
Parts:
- added C405, C406, C408: 100n, Capacitor_SMD:C_0603_1608Metric, symbol Device:C_Small
- added C407: 4.7µ/10V, Capacitor_Tantalum_SMD:CP_EIA-3216-12_Kemet-S, symbol Device:C_Polarized_Small
- added D401, D402: ORANGE, symbol Device:LED
- added L401: 22µ, symbol Device:L_Small
- added R402, R403: 2k2, Resistor_SMD:R_0603_1608Metric, symbol Device:R
- added R404, R406, R407: 0, symbol Device:R
- added R405: NC, Resistor_SMD:R_0603_1608Metric, symbol Device:R
- added R408, R409: 4k7, Resistor_SMD:R_0603_1608Metric, symbol Device:R
- added R410: 120, Resistor_SMD:R_1206_3216Metric, symbol Device:R
- added U402: FT232RL, Package_SO:SSOP-28_5.3x10.2mm_P0.65mm, symbol Interface_USB:FT232RL
- added U403: TJA1051T, Package_SO:SOIC-8_3.9x4.9mm_P1.27mm, symbol Interface_CAN_LIN:TJA1051T
Connections:
- net GND: now also C405.2, C406.2, C407.2, C408.1, R402.2, U402.18 (GND), U402.21 (GND), U402.25 (AGND), U402.26 (TEST), U402.7 (GND), U403.2 (GND), U403.8 (S)
- net RESET: now also R404.2
- net CAN-TX: now reaches U401.4 (SENSOR_VP)
- net CAN-TX: now also U403.1 (TXD)
- net CAN-RX: now reaches U401.5 (SENSOR_VN)
- net CAN-RX: now also U403.4 (RXD)
- new net: R407.1, U402.1 (TXD)
- new net: R404.1, U402.3 (RTS)
- new net: D402.1 (K), R409.2
- new net: R402.1, R403.2, U402.19 (~{RESET})
- new net: R408.1, U402.23 (CBUS0)
- new net: D401.1 (K), R408.2
- new net: R405.1, U402.2 (DTR)
- new net: R409.1, U402.22 (CBUS1)
- new net: C408.2, U402.17 (3V3OUT), U402.4 (VCCIO)
- new net: R406.1, U402.5 (RXD)
- new net +3V3: D401.2 (A), D402.2 (A)
- new net +5VD: C405.1, C406.1, C407.1, L401.2, R403.1, U402.20 (VCC), U403.3 (VCC)
- new net CANH: R410.2, U403.7 (CANH)
- new net CANL: R410.1, U403.6 (CANL)
- new net D+: U402.15 (USBD+)
- new net D-: U402.16 (USBD-)
- new net RXD0: R407.2
- new net TXD0: R406.2
- new net VCCUSB: L401.1
- no-connect marks 0 -> 10
Other:
- company: (none) -> CMOS-74A
- title: (none) -> UART
- moved on the sheet: C401, C402, C403, C404, R401, U401

Commit message: update
Connections:
- net RX0 is gone; now on net RXD0: U401.34 (RXD0/IO3)
- net TX0 is gone; now on net TXD0: U401.35 (TXD0/IO1)
- net PWM2: now reaches U401.10 (IO25)
- net PWM3: now reaches U401.11 (IO26)
- net PWM4: now reaches U401.12 (IO27)
- net SCS: now reaches U401.19 (SCS/CMD)
- net SCK: now reaches U401.20 (SCK/CLK)
- net SDO: now reaches U401.21 (SDO/SD0)
- net SDI: now reaches U401.22 (SDI/SD1)
- net RX1: now reaches U401.27 (IO16)
- net TX1: now reaches U401.28 (IO17)
- net SDA1: now reaches U401.30 (IO18)
- net SCL1: now reaches U401.31 (IO19)
- net RX2: now reaches U401.6 (IO34)
- net TX2: now reaches U401.7 (IO35)
- net PWM0: now reaches U401.8 (IO32)
- net PWM1: now reaches U401.9 (IO33)
Changed lines of the file:
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@@
+	(wire
+		(pts
+			(xy 237.49 93.98) (xy 242.57 93.98)
+		)
+		(stroke
+			(width 0)
+			(type default)
+		)
+	)
 	(wire
 		(pts
@@
 		(pts
 			(xy 73.66 62.23) (xy 80.01 62.23)
-		)
-		(stroke
-			(width 0)
-			(type default)
-		)
-	)
-	(wire
-		(pts
-			(xy 237.49 93.98) (xy 242.57 93.98)
 		)
 		(stroke
@@
 		)
 	)
+	(hierarchical_label "RX1"
+		(shape input)
+		(at 242.57 76.2 0)
+		(effects
+			(font
+				(size 1.27 1.27)
+			)
+			(justify left)
+		)
+	)
+	(hierarchical_label "TX1"
+		(shape input)
+		(at 242.57 78.74 0)
+		(effects
+			(font
+				(size 1.27 1.27)
+			)
+			(justify left)
+		)
+	)
 	(hierarchical_label "CANH"
 		(shape input)
@@
 		)
 	)
+	(hierarchical_label "PWM0"
+		(shape input)
+		(at 242.57 101.6 0)
+		(effects
+			(font
+				(size 1.27 1.27)
+			)
+			(justify left)
+		)
+	)
 	(hierarchical_label "CANL"
 		(shape input)
@@
 		)
 	)
-	(hierarchical_label "RX0"
+	(hierarchical_label "RXD0"
 		(shape input)
 		(at 242.57 58.42 0)
@@
 		)
 	)
-	(hierarchical_label "TX0"
+	(hierarchical_label "SDI"
+		(shape input)
+		(at 201.93 83.82 180)
+		(effects
+			(font
+				(size 1.27 1.27)
+			)
+			(justify right)
+		)
+	)
+	(hierarchical_label "PWM1"
+		(shape input)
+		(at 242.57 104.14 0)
+		(effects
+			(font
+				(size 1.27 1.27)
+			)
+			(justify left)
+		)
+	)
+	(hierarchical_label "TXD0"
 		(shape input)
 		(at 242.57 53.34 0)
@@
 		)
 	)
+	(hierarchical_label "SCS"
+		(shape input)
+		(at 201.93 93.98 180)
+		(effects
+			(font
+				(size 1.27 1.27)
+			)
+			(justify right)
+		)
+	)
+	(hierarchical_label "SDA1"
+		(shape input)
+		(at 242.57 81.28 0)
+		(effects
+			(font
+				(size 1.27 1.27)
+			)
+			(justify left)
+		)
+	)
 	(hierarchical_label "RXD0"
 		(shape input)
@@
 		)
 	)
+	(hierarchical_label "SCL1"
+		(shape input)
+		(at 242.57 83.82 0)
+		(effects
+			(font
+				(size 1.27 1.27)
+			)
+			(justify left)
+		)
+	)
+	(hierarchical_label "RX2"
+		(shape input)
+		(at 242.57 106.68 0)
+		(effects
+			(font
+				(size 1.27 1.27)
+			)
+			(justify left)
+		)
+	)
+	(hierarchical_label "PWM2"
+		(shape input)
+		(at 242.57 93.98 0)
+		(effects
+			(font
+				(size 1.27 1.27)
+			)
+			(justify left)
+		)
+	)
 	(hierarchical_label "SDA"
 		(shape input)
@@
 		)
 	)
+	(hierarchical_label "PWM4"
+		(shape input)
+		(at 242.57 99.06 0)
+		(effects
+			(font
+				(size 1.27 1.27)
+			)
+			(justify left)
+		)
+	)
+	(hierarchical_label "PWM3"
+		(shape input)
+		(at 242.57 96.52 0)
+		(effects
+			(font
+				(size 1.27 1.27)
+			)
+			(justify left)
+		)
+	)
+	(hierarchical_label "TX2"
+		(shape input)
+		(at 242.57 109.22 0)
+		(effects
+			(font
+				(size 1.27 1.27)
+			)
+			(justify left)
+		)
+	)
 	(hierarchical_label "VCCUSB"
 		(shape input)
@@
 		)
 	)
+	(hierarchical_label "SCK"
+		(shape input)
+		(at 201.93 91.44 180)
+		(effects
+			(font
+				(size 1.27 1.27)
+			)
+			(justify right)
+		)
+	)
+	(hierarchical_label "SDO"
+		(shape input)
+		(at 201.93 81.28 180)
+		(effects
+			(font
+				(size 1.27 1.27)
+			)
+			(justify right)
+		)
+	)
