File: KICAD/CPU_ESP/V0.1/CPU/ESP32.kicad_sch (KiCad schematic)
At the start: 30 parts, among them U401 ESP32-WROOM-32, U402 FT232RL, U403 TJA1051T

Commit message: update
Connections:
- net RW: now reaches U401.13 (IO14)
- net E: now reaches U401.16 (IO13)
- net T1CK: now reaches U401.17 (SHD/SD2)
- net T2CK: now reaches U401.18 (SWP/SD3)
- net RS: now reaches U401.23 (IO15)
- net IO8: now reaches U401.37 (IO23)
- net RXD0 renamed RX0
- net TXD0 renamed TX0
Changed lines of the file:
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@@
+		)
+	)
+	(hierarchical_label "IO8"
+		(shape input)
+		(at 195.58 90.17 0)
+		(effects
+			(font
+				(size 1.27 1.27)
+			)
+			(justify left)
 		)
 	)
@@
 		)
 	)
+	(hierarchical_label "RW"
+		(shape input)
+		(at 195.58 69.85 0)
+		(effects
+			(font
+				(size 1.27 1.27)
+			)
+			(justify left)
+		)
+	)
 	(hierarchical_label "TX1"
 		(shape input)
@@
 		)
 	)
+	(hierarchical_label "E"
+		(shape input)
+		(at 195.58 67.31 0)
+		(effects
+			(font
+				(size 1.27 1.27)
+			)
+			(justify left)
+		)
+	)
+	(hierarchical_label "T2CK"
+		(shape input)
+		(at 154.94 87.63 180)
+		(effects
+			(font
+				(size 1.27 1.27)
+			)
+			(justify right)
+		)
+	)
 	(hierarchical_label "D+"
 		(shape input)
@@
 		)
 	)
-	(hierarchical_label "TXD0"
+	(hierarchical_label "TX0"
 		(shape input)
 		(at 123.19 140.97 0)
@@
 		)
 	)
-	(hierarchical_label "RXD0"
+	(hierarchical_label "RX0"
 		(shape input)
 		(at 195.58 57.15 0)
@@
 		)
 	)
-	(hierarchical_label "TXD0"
+	(hierarchical_label "TX0"
 		(shape input)
 		(at 195.58 52.07 0)
@@
 		)
 	)
-	(hierarchical_label "RXD0"
+	(hierarchical_label "RX0"
 		(shape input)
 		(at 123.19 138.43 0)
@@
 		)
 	)
+	(hierarchical_label "RS"
+		(shape input)
+		(at 195.58 72.39 0)
+		(effects
+			(font
+				(size 1.27 1.27)
+			)
+			(justify left)
+		)
+	)
 	(hierarchical_label "SDA"
 		(shape input)
@@
 		)
 	)
+	(hierarchical_label "T1CK"
+		(shape input)
+		(at 154.94 85.09 180)
+		(effects
+			(font
+				(size 1.27 1.27)
+			)
+			(justify right)
+		)
+	)

Commit message: update
Parts:
- D401, D402: footprint (none) -> LED_SMD:LED_0603_1608Metric
- L401: footprint (none) -> Inductor_SMD:L_1008_2520Metric
- R404, R406, R407: footprint (none) -> Resistor_SMD:R_0603_1608Metric
Changed lines of the file:
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@@
 			)
 		)
-		(property "Footprint" ""
+		(property "Footprint" "Resistor_SMD:R_0603_1608Metric"
 			(at 110.49 140.208 90)
 			(effects
@@
 		)
 		(property "Description" "Resistor"
+			(at 110.49 138.43 0)
+			(effects
+				(font
+					(size 1.27 1.27)
+				)
+				(hide yes)
+			)
+		)
+		(property "UART" ""
 			(at 110.49 138.43 0)
 			(effects
@@
 			)
 		)
-		(property "Footprint" ""
+		(property "Footprint" "Resistor_SMD:R_0603_1608Metric"
 			(at 110.49 145.288 90)
 			(effects
@@
 		)
 		(property "Description" "Resistor"
+			(at 110.49 143.51 0)
+			(effects
+				(font
+					(size 1.27 1.27)
+				)
+				(hide yes)
+			)
+		)
+		(property "UART" ""
 			(at 110.49 143.51 0)
 			(effects
@@
 			)
 		)
-		(property "Footprint" ""
+		(property "Footprint" "LED_SMD:LED_0603_1608Metric"
 			(at 132.08 160.02 0)
 			(effects
@@
 		)
 		(property "Sim.Pins" "1=K 2=A"
+			(at 132.08 160.02 0)
+			(effects
+				(font
+					(size 1.27 1.27)
+				)
+				(hide yes)
+			)
+		)
+		(property "UART" ""
 			(at 132.08 160.02 0)
 			(effects
@@
 			)
 		)
+		(property "UART" ""
+			(at 110.49 148.59 0)
+			(effects
+				(font
+					(size 1.27 1.27)
+				)
+				(hide yes)
+			)
+		)
 		(pin "1"
 		)
@@
 			)
 		)
-		(property "Footprint" ""
+		(property "Footprint" "LED_SMD:LED_0603_1608Metric"
 			(at 120.65 160.02 0)
 			(effects
@@
 		)
 		(property "Sim.Pins" "1=K 2=A"
+			(at 120.65 160.02 0)
+			(effects
+				(font
+					(size 1.27 1.27)
+				)
+				(hide yes)
+			)
+		)
+		(property "UART" ""
 			(at 120.65 160.02 0)
 			(effects
@@
 			)
 		)
-		(property "Footprint" ""
+		(property "Footprint" "Inductor_SMD:L_1008_2520Metric"
 			(at 29.21 156.21 0)
 			(effects
@@
 			)
 		)
+		(property "UART" ""
+			(at 29.21 156.21 0)
+			(effects
+				(font
+					(size 1.27 1.27)
+				)
+				(hide yes)
+			)
+		)
 		(pin "2"
 		)
@@
 			)
 		)
-		(property "Footprint" ""
+		(property "Footprint" "Resistor_SMD:R_0603_1608Metric"
 			(at 110.49 142.748 90)
 			(effects
@@
 			(at 110.49 140.97 0)
 			(effects
+				(font
+					(size 1.27 1.27)
+				)
+				(hide yes)
+			)
+		)
+		(property "UART" ""
+			(at 110.49 140.97 0)
+			(effects

Commit message: PCB update
Connections:
- net IO8: now also U401.6 (IO34); no longer U401.37 (IO23)
- net RX2: now also U401.17 (SHD/SD2); no longer U401.6 (IO34)
- net T1CK: now also U401.37 (IO23); no longer U401.17 (SHD/SD2)
- net T2CK: now also U401.29 (IO5); no longer U401.18 (SWP/SD3)
- net TX2: now also U401.18 (SWP/SD3); no longer U401.7 (IO35)
- net at R413.2: now also U401.7 (IO35); no longer U401.29 (IO5)

Commit message: PCB to control
Connections:
- net +3V3 is gone; now on net +3.3V: D401.2 (A), D402.2 (A)

Commit message: KICADUpdate
Parts:
- C402: value 22µ/10V -> 10µ/10V
- C407: value 4.7µ/10V -> 10µ/10V
Changed lines of the file:
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@@
 			)
 		)
-		(property "Value" "22µ/10V"
+		(property "Value" "10µ/10V"
 			(at 140.97 29.21 0)
 			(effects
@@
 			)
 		)
-		(property "Value" "4.7µ/10V"
+		(property "Value" "10µ/10V"
 			(at 107.95 120.1038 0)
 			(effects
