File: KICAD/CPU_ESP/V0.1/CPU/I2C.kicad_sch (KiCad schematic)
At the start: 0 parts

Commit message: Update
Parts:
- added C201: C, symbol Device:C
- added C202, C203: C_Polarized, symbol Device:C_Polarized
- added D201: D_Schottky, symbol Device:D_Schottky
- added R201: R, symbol Device:R
- added U201: PCF8563T, Package_SO:SOIC-8_3.9x4.9mm_P1.27mm, symbol Timer_RTC:PCF8563T
- added U202: LM75C, symbol Sensor_Temperature:LM75C
- added U203: PCA9306, symbol Interface:PCA9306
- added U204: TCA9544A, Package_SO:TSSOP-20_4.4x6.5mm_P0.65mm, symbol Interface_Expansion:TCA9544A
- added U206: TCA9548APWR, Package_SO:TSSOP-24_4.4x7.8mm_P0.65mm, symbol Interface_Expansion:TCA9548APWR
- added U207: P82B715, Package_SO:SO-8_3.9x4.9mm_P1.27mm, symbol CMOS-LIBRAIRIE:P82B715
- added Y201: Crystal_Small, symbol Device:Crystal_Small
Connections:
- new net: C201.1, U201.2 (OSCO), Y201.1
- new net: D201.1 (K), R201.1, U201.8 (VDD)
- new net: C202.1, R201.2
- new net: C202.2, C203.1
- new net: U201.1 (OSCI), Y201.2
- new net GND: C201.2, C203.2, U201.4 (VSS)
- no-connect marks 0 -> 2

Commit message: Update
Parts:
- removed U207: P82B715, Package_SO:SO-8_3.9x4.9mm_P1.27mm, symbol CMOS-LIBRAIRIE:P82B715
- added D202: RED, symbol Device:LED
- added R202: 330, symbol Device:R
- added R203, R204, R205, R206: 2.2K, symbol Device:R
- added R207, R209, R211: NC, symbol Device:R
- added R208, R210, R212: 0, symbol Device:R
- C202, C203: value C_Polarized -> 10F/2.7V
- R201: value R -> 150
- U202: value LM75C -> LM75A
- Y201: value Crystal_Small -> 32.768Khz
Connections:
- net GND: now also U202.4 (GND), U202.5 (A2), U202.6 (A1), U202.7 (A0), U203.1 (GND), R208.2, R210.2, R212.2
- net +5VD: now reaches D201.2 (A)
- net +5VD: now also U202.8 (+Vs), U203.7 (VREF2), U203.8 (EN), R205.1, R206.1
- net SDA-5V: now reaches U202.1 (SDA)
- net SDA-5V: now also U201.5 (SDA), U203.5 (SDA2), R206.2
- net SCL-5V: now reaches U202.2 (SCL)
- net SCL-5V: now also U201.6 (SCL), U203.6 (SCL2), R205.2
- net at U202.3 (O.S.): now also R202.2
- net +3.3V: now reaches U203.2 (VREF1)
- net +3.3V: now also D202.2 (A), R203.1, R204.1, R207.1, R209.1, R211.1
- net SCL0: now reaches U203.3 (SCL1)
- net SCL0: now also U204.18 (SCL), U206.22 (SCL), R203.2
- net SDA0: now reaches U203.4 (SDA1)
- net SDA0: now also U204.19 (SDA), U206.23 (SDA), R204.2
- net at U206.1 (A0): now also R211.2, R212.1
- net at U206.2 (A1): now also R209.2, R210.1
- net at U206.21 (A2): now also R207.2, R208.1
- net RST: now reaches U206.3 (~{RESET})
- new net: D202.1 (K), R202.1
Other:
- note added: "REAL TIME CLOCK"
- moved on the sheet: C201, C202, C203, D201, R201, U201, U202, U203, U204, U206, Y201

Commit message: Update
Parts:
- removed U206: TCA9548APWR, Package_SO:TSSOP-24_4.4x7.8mm_P0.65mm, symbol Interface_Expansion:TCA9548APWR
- added R213, R215, R217: NC, symbol Device:R
- added R214, R216, R218: 0, symbol Device:R
- added U205: MCP23017_SO, Package_SO:SOIC-28W_7.5x17.9mm_P1.27mm, symbol Interface_Expansion:MCP23017_SO
- added U206: AT24CS01-MAHM, Package_DFN_QFN:DFN-8-1EP_3x2mm_P0.5mm_EP1.3x1.5mm, symbol Memory_EEPROM:AT24CS01-MAHM
Connections:
- net SDA-5V is gone; now on net SCL-5V: R206.2, U201.5 (SDA), U202.1 (SDA), U203.5 (SDA2)
- net +3.3V: now also U204.20 (VCC), R213.1, R215.1, R217.1, U205.9 (VDD)
- net GND: now also U204.10 (GND), R214.2, R216.2, R218.2, U205.10 (VSS), U206.1 (A0), U206.2 (A1), U206.3 (A2), U206.4 (GND), U206.9 (GND)
- net RST: now also U205.18 (~{RESET})
- net SCL0: now also U204.6 (SC0); no longer R203.2, U203.3 (SCL1), U204.18 (SCL)
- net SDA0: now also U204.5 (SD0); no longer R204.2, U203.4 (SDA1), U204.19 (SDA)
- net at R207.2, R208.1: now also U205.17 (A2)
- net at R211.2, R212.1: now also U205.15 (A0)
- net at R209.2, R210.1: now also U205.16 (A1)
- net at U204.1 (A0): now also R213.2, R214.1
- net SDA2: now reaches U204.12 (SD2)
- net SCL2: now reaches U204.13 (SC2)
- net SDA3: now reaches U204.15 (SD3)
- net SCL3: now reaches U204.16 (SC3)
- net at U204.2 (A1): now also R215.2, R216.1
- net at U204.3 (A2): now also R217.2, R218.1
- net SDA1: now reaches U204.8 (SD1)
- net SCL1: now reaches U204.9 (SC1)
- new net D0: U205.1 (GPB0)
- new net D1: U205.2 (GPB1)
- new net D2: U205.3 (GPB2)
- new net D3: U205.4 (GPB3)
- new net D4: U205.5 (GPB4)
- new net D5: U205.6 (GPB5)
- new net D6: U205.7 (GPB6)
- new net D7: U205.8 (GPB7)
- new net IO0: U205.21 (GPA0)
- new net IO1: U205.22 (GPA1)
- new net IO2: U205.23 (GPA2)
- new net IO3: U205.24 (GPA3)
- new net IO4: U205.25 (GPA4)
- new net IO5: U205.26 (GPA5)
- new net IO6: U205.27 (GPA6)
- new net IO7: U205.28 (GPA7)
- new net SCL: R203.2, U203.3 (SCL1), U204.18 (SCL), U205.13 (SDA)
- new net SDA: R204.2, U203.4 (SDA1), U204.19 (SDA), U205.12 (SCK)
- no-connect marks 2 -> 10
Other:
- moved on the sheet: R207, R208, R209, R210, R211, R212, U204

Commit message: Update
Parts:
- D201: footprint (none) -> Diode_SMD:D_1206_3216Metric
- R201, R202, R203, R204, R205, R206, R207, R208, R209, R210, R211, R212, R213, R214, R215, R216, R217, R218: footprint (none) -> Resistor_SMD:R_0603_1608Metric
Connections:
- net +5VD: now also U206.8 (VCC)
- net SCL-5V: now also U206.5 (SDA), U206.6 (SCL)

Commit message: Update
Parts:
- added R105, R106, R109, R110, R111, R112, R113, R114: 2.2k, Resistor_SMD:R_0603_1608Metric, symbol Device:R
- C201: footprint (none) -> Capacitor_SMD:C_0603_1608Metric
- C202, C203: footprint (none) -> Capacitor_THT:CP_Radial_Tantal_D5.0mm_P5.00mm
- D202: footprint (none) -> LED_SMD:LED_0603_1608Metric
- U202: footprint (none) -> Package_SO:SOIC-8_3.9x4.9mm_P1.27mm
- U203: footprint (none) -> Package_SO:VSSOP-8_2.3x2mm_P0.5mm
- Y201: footprint (none) -> Crystal:Crystal_SMD_TXC_9HT11-2Pin_2.0x1.2mm
Connections:
- net +3.3V: now also R105.1, R106.1, R109.1, R110.1, R111.1, R112.1, R113.1, R114.1
- net SCL0: now also R111.2
- net SCL1: now also R109.2
- net SCL2: now also R105.2, R106.2
- net SCL3: now also R113.2
- net SDA0: now also R112.2
- net SDA1: now also R110.2
- net SDA3: now also R114.2
- net RST renamed RESET
Other:
- moved on the sheet: U206

Commit message: update
Parts:
- added U207: PCA9531PW, Package_SO:TSSOP-16_4.4x5mm_P0.65mm, symbol Driver_LED:PCA9531PW
Connections:
- net +5VD: now also U207.16 (V_{DD})
- net GND: now also U207.1 (A0), U207.2 (A1), U207.3 (A2), U207.8 (V_{SS})
- net RESET: now also U207.13 (~{RESET})
- net SCL-5V: now also U207.14 (SCL), U207.15 (SDA)
- new net PWM0: U207.4 (LED0)
- new net PWM1: U207.5 (LED1)
- new net PWM2: U207.6 (LED2)
- new net PWM3: U207.7 (LED3)
- new net PWM4: U207.9 (LED4)
- new net PWM5: U207.10 (LED5)
- new net PWM6: U207.11 (LED6)
- new net PWM7: U207.12 (LED7)
Other:
- company: (none) -> CMOS-74A
- title: (none) -> I2C

Commit message: update
Parts:
- removed R207, R209, R211, R213, R215, R217: NC, Resistor_SMD:R_0603_1608Metric, symbol Device:R
- removed U207: PCA9531PW, Package_SO:TSSOP-16_4.4x5mm_P0.65mm, symbol Driver_LED:PCA9531PW
- renumbered C202 to C204, C203 to C205, C201 to C206, D201 to D203, D202 to D204, R105 to R107, R106 to R108, R111 to R115, R112 to R116, R109 to R117, R110 to R118, R113 to R119, R114 to R120, R201 to R207, R204 to R209, R203 to R211, R202 to R213, R205 to R215, R206 to R217, R214 to R219, R212 to R220, R216 to R221, R210 to R222, R218 to R223, R208 to R224, U202 to U208, U203 to U209, U201 to U210, U204 to U212, U205 to U213, U206 to U214, Y201 to Y202
Connections:
- net SCL: no longer U212.18 (SCL)
- net SCL1: now also U212.18 (SCL); no longer R117.2, U212.9 (SC1)
- net SDA: no longer U212.19 (SDA)
- net SDA1: now also U212.19 (SDA); no longer R118.2, U212.8 (SD1)
- net SCL0 renamed SCL0-E
- net SCL2 renamed SCL2-E
- net SCL3 renamed SCL3-E
- net SDA0 renamed SDA0-E
- net SDA2 renamed SDA2-E
- net SDA3 renamed SDA3-E
- new net SCL1-E: R117.2, U212.9 (SC1)
- new net SDA1-E: R118.2, U212.8 (SD1)
