File: KICAD/CPU_ESP/V0.1/CPU/I2C.kicad_sch (KiCad schematic)
At the start: 32 parts, among them U201 LM75A, U202 PCA9306, U203 PCF8563T, U204 TCA9544A, U205 MCP23017_SO, U206 AT24CS01-MAHM, Y201 32.278kHz

Commit message: update
Parts:
- removed U206: AT24CS01-MAHM, Package_SO:SOIC-8_5.3x5.3mm_P1.27mm, symbol Memory_EEPROM:AT24CS01-MAHM
- added U207: AT24CS01-SSHM, Package_SO:SOIC-8_5.3x5.3mm_P1.27mm, symbol Memory_EEPROM:AT24CS01-SSHM
Connections:
- net +5VD: now also U207.8 (VCC)
- net GND: now also U207.1 (A0), U207.2 (A1), U207.3 (A2), U207.4 (GND)
- net SCL-5V: now also U207.6 (SCL)
- net SDA-5V: now also U207.5 (SDA)
Changed lines of the file:
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@@
-	)
-	(symbol
-		(lib_id "Memory_EEPROM:AT24CS01-MAHM")
-		(at 256.54 90.17 0)
-		(unit 1)
-		(exclude_from_sim no)
-		(in_bom yes)
-		(on_board yes)
-		(dnp no)
-		(fields_autoplaced yes)
-		(property "Reference" "U206"
-			(at 258.6833 80.01 0)
-			(effects
-				(font
-					(size 1.27 1.27)
-				)
-				(justify left)
-			)
-		)
-		(property "Value" "AT24CS01-MAHM"
-			(at 258.6833 82.55 0)
-			(effects
-				(font
-					(size 1.27 1.27)
-				)
-				(justify left)
-			)
-		)
-		(property "Footprint" "Package_SO:SOIC-8_5.3x5.3mm_P1.27mm"
-			(at 256.54 90.17 0)
-			(effects
-				(font
-					(size 1.27 1.27)
-				)
-				(hide yes)
-			)
-		)
-		(property "Datasheet" "http://ww1.microchip.com/downloads/en/DeviceDoc/Atmel-8815-SEEPROM-AT24CS01-02-Datasheet.pdf"
-			(at 256.54 90.17 0)
-			(effects
-				(font
-					(size 1.27 1.27)
-				)
-				(hide yes)
-			)
-		)
-		(property "Description" "I2C Serial EEPROM, 1Kb (128x8) with Unique Serial Number, UDFN8"
-			(at 256.54 90.17 0)
-			(effects
-				(font
-					(size 1.27 1.27)
-				)
-				(hide yes)
-			)
-		)
-		(property "UART" ""
-			(at 256.54 90.17 0)
-			(effects
-				(font
-					(size 1.27 1.27)
-				)
-				(hide yes)
-			)
-		)
-		(pin "5"
-		)
-		(pin "8"
-		)
-		(pin "1"
-		)
-		(pin "4"
-		)
-		(pin "6"
-		)
-		(pin "7"
-		)
-		(pin "9"
-		)
-		(pin "2"
-		)
-		(pin "3"
-		)
-		(instances
-			(project "CPU"
-				(path "/a676c576-12a0-418f-9fc1-1ecc8cb5a083/ebcf0d9a-523d-4f37-81f9-63d54b289420"
-					(reference "U206")
-					(unit 1)
-				)
-			)
-		)
 	)
 	(symbol
@@
 					(unit 1)
 				)
+			)
+		)
+	)
+	(symbol
+		(lib_id "Memory_EEPROM:AT24CS01-SSHM")
+		(at 256.54 90.17 0)
+		(unit 1)
+		(exclude_from_sim no)
+		(in_bom yes)
+		(on_board yes)
+		(dnp no)
+		(fields_autoplaced yes)
+		(property "Reference" "U207"
+			(at 258.6833 80.01 0)
+			(effects
+				(font
+					(size 1.27 1.27)
+				)
+				(justify left)
+			)
+		)
+		(property "Value" "AT24CS01-SSHM"
+			(at 258.6833 82.55 0)
+			(effects
+				(font
+					(size 1.27 1.27)
+				)
+				(justify left)
+			)
+		)
+		(property "Footprint" "Package_SO:SOIC-8_5.3x5.3mm_P1.27mm"
+			(at 256.54 90.17 0)
+			(effects
+				(font
+					(size 1.27 1.27)
+				)
+				(hide yes)
+			)
+		)
+		(property "Datasheet" "http://ww1.microchip.com/downloads/en/DeviceDoc/Atmel-8815-SEEPROM-AT24CS01-02-Datasheet.pdf"
+			(at 256.54 90.17 0)
+			(effects
+				(font
+					(size 1.27 1.27)
+				)
+				(hide yes)
+			)
+		)
+		(property "Description" "I2C Serial EEPROM, 1Kb (128x8) with Unique Serial Number, SO8"
+			(at 256.54 90.17 0)
+			(effects
+				(font
+					(size 1.27 1.27)
+				)
+				(hide yes)
+			)
+		)
+		(property "UART" ""
+			(at 256.54 90.17 0)
+			(effects
+				(font
+					(size 1.27 1.27)
+				)
+				(hide yes)
+			)
+		)
+		(pin "7"
+		)
+		(pin "2"
+		)
+		(pin "4"
+		)
+		(pin "8"
+		)
+		(pin "6"
+		)
+		(pin "1"
+		)
+		(pin "3"
+		)
+		(pin "5"
+		)
+		(instances
+			(project ""
+				(path "/a676c576-12a0-418f-9fc1-1ecc8cb5a083/ebcf0d9a-523d-4f37-81f9-63d54b289420"
+					(reference "U207")
+					(unit 1)
+				)

Commit message: update
Parts:
- removed R105, R106, R109, R110, R111, R112, R113, R114: 2.2k, Resistor_SMD:R_0603_1608Metric, symbol Device:R
- added R208, R209, R211, R213, R215, R217: 2k2, Resistor_SMD:R_0603_1608Metric_Pad0.98x0.95mm_HandSolder, symbol Device:R
Connections:
- net +3.3V: now also R208.1, R209.1, R211.1, R213.1, R215.1, R217.1
- net SCL0-E: now also R208.2
- net SCL1-E: now also R211.2
- net SCL2-E: now also R215.2
- net SDA0-E: now also R209.2
- net SDA1-E: now also R213.2
- net SDA2-E: now also R217.2
- net SCL3-E: no longer names the net of U204.16 (SC3)
- net SDA3-E: no longer names the net of U204.15 (SD3)
- no-connect marks 12 -> 14

Commit message: PCB update
Parts:
- added R219, R220: 2k2, Resistor_SMD:R_0603_1608Metric, symbol Device:R
Connections:
- net +3.3V: now also R219.1, R220.1
- net SCL1: now also R219.2
- net SDA1: now also R220.2

Commit message: PCB to control
Parts:
- removed U205: MCP23017_SO, Package_SO:SOIC-28W_7.5x17.9mm_P1.27mm, symbol Interface_Expansion:MCP23017_SO
- added U205: MCP23017_SS, Package_SO:SSOP-28_5.3x10.2mm_P0.65mm, symbol Interface_Expansion:MCP23017_SS
Connections:
- net +3.3V: now also U205.9 (VDD)
- net D0: now also U205.1 (GPB0)
- net D1: now also U205.2 (GPB1)
- net D2: now also U205.3 (GPB2)
- net D3: now also U205.4 (GPB3)
- net D4: now also U205.5 (GPB4)
- net D5: now also U205.6 (GPB5)
- net D6: now also U205.7 (GPB6)
- net D7: now also U205.8 (GPB7)
- net GND: now also U205.10 (VSS)
- net IO0: now also U205.21 (GPA0)
- net IO1: now also U205.22 (GPA1)
- net IO2: now also U205.23 (GPA2)
- net IO3: now also U205.24 (GPA3)
- net IO4: now also U205.25 (GPA4)
- net IO5: now also U205.26 (GPA5)
- net IO6: now also U205.27 (GPA6)
- net IO7: now also U205.28 (GPA7)
- net RESET: now also U205.18 (~{RESET})
- net SCL: now also U205.12 (SCK)
- net SDA: now also U205.13 (SDA)
- net at R210.1: now also U205.16 (A1)
- net at R212.1: now also U205.15 (A0)
- net at R207.1: now also U205.17 (A2)
Changed lines of the file:
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@@
+	)
+	(symbol
+		(lib_id "Interface_Expansion:MCP23017_SS")
+		(at 193.04 128.27 0)
+		(unit 1)
+		(exclude_from_sim no)
+		(in_bom yes)
+		(on_board yes)
+		(dnp no)
+		(fields_autoplaced yes)
+		(property "Reference" "U205"
+			(at 195.1833 100.33 0)
+			(effects
+				(font
+					(size 1.27 1.27)
+				)
+				(justify left)
+			)
+		)
+		(property "Value" "MCP23017_SS"
+			(at 195.1833 102.87 0)
+			(effects
+				(font
+					(size 1.27 1.27)
+				)
+				(justify left)
+			)
+		)
+		(property "Footprint" "Package_SO:SSOP-28_5.3x10.2mm_P0.65mm"
+			(at 198.12 153.67 0)
+			(effects
+				(font
+					(size 1.27 1.27)
+				)
+				(justify left)
+				(hide yes)
+			)
+		)
+		(property "Datasheet" "https://ww1.microchip.com/downloads/aemDocuments/documents/APID/ProductDocuments/DataSheets/MCP23017-Data-Sheet-DS20001952.pdf"
+			(at 198.12 156.21 0)
+			(effects
+				(font
+					(size 1.27 1.27)
+				)
+				(justify left)
+				(hide yes)
+			)
+		)
+		(property "Description" "16-bit I/O expander, I2C, interrupts, w pull-ups, SSOP-28"
+			(at 193.04 128.27 0)
+			(effects
+				(font
+					(size 1.27 1.27)
+				)
+				(hide yes)
+			)
+		)
+		(pin "2"
+		)
+		(pin "25"
+		)
+		(pin "3"
+		)
+		(pin "27"
+		)
+		(pin "16"
+		)
+		(pin "22"
+		)
+		(pin "21"
+		)
+		(pin "15"
+		)
+		(pin "24"
+		)
+		(pin "28"
+		)
+		(pin "14"
+		)
+		(pin "23"
+		)
+		(pin "11"
+		)
+		(pin "26"
+		)
+		(pin "6"
+		)
+		(pin "5"
+		)
+		(pin "4"
+		)
+		(pin "1"
+		)
+		(pin "19"
+		)
+		(pin "17"
+		)
+		(pin "18"
+		)
+		(pin "20"
+		)
+		(pin "12"
+		)
+		(pin "9"
+		)
+		(pin "13"
+		)
+		(pin "7"
+		)
+		(pin "8"
+		)
+		(pin "10"
+		)
+		(instances
+			(project ""
+				(path "/a676c576-12a0-418f-9fc1-1ecc8cb5a083/ebcf0d9a-523d-4f37-81f9-63d54b289420"
+					(reference "U205")
+					(unit 1)
+				)
+			)
+		)
 	)
 	(symbol
@@
 					(unit 1)
 				)
-			)
-		)
-	)
-	(symbol
-		(lib_id "Interface_Expansion:MCP23017_SO")
-		(at 193.04 128.27 0)
-		(unit 1)
-		(exclude_from_sim no)
-		(in_bom yes)
-		(on_board yes)
-		(dnp no)
-		(fields_autoplaced yes)
-		(property "Reference" "U205"
-			(at 195.1833 100.33 0)
-			(effects
-				(font
-					(size 1.27 1.27)
-				)
-				(justify left)
-			)
-		)
-		(property "Value" "MCP23017_SO"
-			(at 195.1833 102.87 0)
-			(effects
-				(font
-					(size 1.27 1.27)
-				)
-				(justify left)
-			)
-		)
-		(property "Footprint" "Package_SO:SOIC-28W_7.5x17.9mm_P1.27mm"
-			(at 198.12 153.67 0)
-			(effects
-				(font
-					(size 1.27 1.27)
-				)
-				(justify left)
-				(hide yes)
-			)
-		)
-		(property "Datasheet" "https://ww1.microchip.com/downloads/aemDocuments/documents/APID/ProductDocuments/DataSheets/MCP23017-Data-Sheet-DS20001952.pdf"
-			(at 198.12 156.21 0)
-			(effects
-				(font
-					(size 1.27 1.27)
-				)
-				(justify left)
-				(hide yes)
-			)
-		)
-		(property "Description" "16-bit I/O expander, I2C, interrupts, w pull-ups, GPA/B7 output only (https://microchip.my.site.com/s/article/GPA7---GPB7-Cannot-Be-Used-as-Inputs-In-MCP23017),  SOIC-28"
-			(at 193.04 128.27 0)
-			(effects
-				(font
-					(size 1.27 1.27)
-				)
-				(hide yes)
-			)
-		)
-		(pin "26"
-		)
-		(pin "13"
-		)
-		(pin "24"
-		)
-		(pin "15"
-		)
-		(pin "8"
-		)
-		(pin "18"
-		)
-		(pin "23"
-		)
-		(pin "14"
-		)
-		(pin "20"
-		)
-		(pin "7"
-		)
-		(pin "19"
-		)
-		(pin "12"
-		)
-		(pin "25"
-		)
-		(pin "5"
-		)
-		(pin "1"
-		)
-		(pin "3"
-		)
-		(pin "4"
-		)
-		(pin "17"
-		)
-		(pin "28"
-		)
-		(pin "11"
-		)
-		(pin "2"
-		)
-		(pin "21"
-		)
-		(pin "22"
-		)
-		(pin "10"
-		)
-		(pin "16"
-		)
-		(pin "6"
-		)
-		(pin "27"
-		)
-		(pin "9"
-		)
-		(instances
-			(project "CPU"
-				(path "/a676c576-12a0-418f-9fc1-1ecc8cb5a083/ebcf0d9a-523d-4f37-81f9-63d54b289420"
-					(reference "U205")
-					(unit 1)
-				)

Commit message: PCB Update
Parts:
- U203: footprint Package_SO:SOIC-8_3.9x4.9mm_P1.27mm -> Package_SO:MSOP-8_3x3mm_P0.65mm
Changed lines of the file:
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@@
 			)
 		)
-		(property "Footprint" "Package_SO:SOIC-8_3.9x4.9mm_P1.27mm"
+		(property "Footprint" "Package_SO:MSOP-8_3x3mm_P0.65mm"
 			(at 55.88 46.99 0)
 			(effects
@@
 			(at 55.88 46.99 0)
 			(effects
+				(font
+					(size 1.27 1.27)
+				)
+				(hide yes)
+			)
+		)
+		(property "UART" ""
+			(at 55.88 46.99 0)
+			(effects
