File: KICAD/CPU_ESP/V0.1/CPU/CPU.kicad_sch (KiCad schematic)
At the start: 3 parts, among them J1 USB_B_Mini, SW2 SW_Push_45deg, SW3 SW_Push_45deg

Commit message: Update
Parts:
- J101: renamed from J1; footprint (none) -> Connector_USB:USB_Mini-B_Wuerth_65100516121_Horizontal
- SW101: renamed from SW2; footprint (none) -> Button_Switch_THT:SW_Tactile_SKHH_Angled
- SW102: renamed from SW3; footprint (none) -> Button_Switch_THT:SW_Tactile_SKHH_Angled
Other:
- added sheet CMOS_BUS (cmos_bus.kicad_sch)
Changed lines of the file:
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@@
 		(dnp no)
 		(fields_autoplaced yes)
-		(property "Reference" "J1"
+		(property "Reference" "J101"
 			(at 31.75 30.48 0)
 			(effects
@@
 			)
 		)
-		(property "Footprint" ""
+		(property "Footprint" "Connector_USB:USB_Mini-B_Wuerth_65100516121_Horizontal"
 			(at 35.56 44.45 0)
 			(effects
@@
 			)
 		)
+		(property "TITLE" ""
+			(at 31.75 43.18 0)
+			(effects
+				(font
+					(size 1.27 1.27)
+				)
+				(hide yes)
+			)
+		)
 		(pin "4"
 		)
@@
 			(project ""
 				(path "/a676c576-12a0-418f-9fc1-1ecc8cb5a083"
-					(reference "J1")
+					(reference "J101")
 					(unit 1)
 				)
@@
 		(dnp no)
 		(fields_autoplaced yes)
-		(property "Reference" "SW3"
+		(property "Reference" "SW102"
 			(at 50.8 121.9199 90)
 			(effects
@@
 			)
 		)
-		(property "Footprint" ""
+		(property "Footprint" "Button_Switch_THT:SW_Tactile_SKHH_Angled"
 			(at 46.99 123.19 0)
 			(effects
@@
 			)
 		)
+		(property "TITLE" ""
+			(at 46.99 123.19 0)
+			(effects
+				(font
+					(size 1.27 1.27)
+				)
+				(hide yes)
+			)
+		)
 		(pin "1"
 		)
@@
 			(project ""
 				(path "/a676c576-12a0-418f-9fc1-1ecc8cb5a083"
-					(reference "SW3")
+					(reference "SW102")
 					(unit 1)
 				)
@@
 		(dnp no)
 		(fields_autoplaced yes)
-		(property "Reference" "SW2"
+		(property "Reference" "SW101"
 			(at 50.8 104.1399 90)
 			(effects
@@
 			)
 		)
-		(property "Footprint" ""
+		(property "Footprint" "Button_Switch_THT:SW_Tactile_SKHH_Angled"
 			(at 46.99 105.41 0)
 			(effects
@@
 			)
 		)
+		(property "TITLE" ""
+			(at 46.99 105.41 0)
+			(effects
+				(font
+					(size 1.27 1.27)
+				)
+				(hide yes)
+			)
+		)
 		(pin "1"
 		)
@@
 			(project ""
 				(path "/a676c576-12a0-418f-9fc1-1ecc8cb5a083"
-					(reference "SW2")
+					(reference "SW101")
 					(unit 1)
 				)
@@
 				)
 			)
+		)
+	)
+	(sheet
+		(at 82.55 101.6)
+		(size 25.4 41.91)
+		(exclude_from_sim no)
+		(in_bom yes)
+		(on_board yes)
+		(dnp no)
+		(fields_autoplaced yes)
+		(stroke
+			(width 0.1524)
+			(type solid)
+		)
+		(fill
+			(color 0 0 0 0.0000)
+		)
+		(property "Sheetname" "CMOS_BUS"
+			(at 82.55 100.8884 0)
+			(effects
+				(font
+					(size 1.27 1.27)
+				)
+				(justify left bottom)
+			)
+		)
+		(property "Sheetfile" "cmos_bus.kicad_sch"
+			(at 82.55 144.0946 0)
+			(effects
+				(font
+					(size 1.27 1.27)
+				)
+				(justify left top)
+			)
+		)
+		(instances
+			(project "CPU"
+				(path "/a676c576-12a0-418f-9fc1-1ecc8cb5a083"
+					(page "5")
+				)
+			)

Commit message: Update
Parts:
- added J102: Conn_01x04, symbol Connector_Generic:Conn_01x04
Connections:
- new net +5VD: J102.2 (Pin_2)
- new net GND: J102.1 (Pin_1)
- new net SCL-5V: J102.3 (Pin_3)
- new net SDA-5V: J102.4 (Pin_4)
Other:
- sheet I2C_Peripherique ports: added RST, SCL-5V, SCL0, SDA-5V, SDA0; removed none

Commit message: Update
Other:
- sheet I2C_Peripherique ports: added D0, D1, D2, D3, D4, D5, D6, D7, IO0, IO1, IO2, IO3, IO4, IO5, IO6, IO7, SCL, SCL1, SCL2, SCL3, SDA, SDA1, SDA2, SDA3; removed none
- moved on the sheet: J102

Commit message: Update
Parts:
- J102: footprint (none) -> Connector_Harwin:Harwin_M20-89004xx_1x04_P2.54mm_Horizontal
Connections:
- no-connect marks 0 -> 1
Other:
- sheet CMOS_BUS ports: added CANRX, CANTX, D0, D1, D2, D3, D4, D5, D6, D7, E, INT0, INT1, IO0, IO1, IO2, IO3, IO4, IO5, IO6, IO7, IO8, IO9, PWM0, PWM1, PWM2, PWM3, PWM4, RESET, RETRO, RS, RW, SCK, SCL0, SCL1, SCL2, SCS, SDA0, SDA1, SDA2, SDI, SDO, T1CK, T2CK, UART-RX0, UART-RX1, UART-RX2, UART-RX3, UART-TX0, UART-TX1, UART-TX2, UART-TX3; removed none
- sheet ESP32 Module ports: added BOOT, RESET, RX0, SCL, SDA, TX0; removed none
- sheet I2C_Peripherique ports: added RESET; removed RST
- moved on the sheet: J102, SW101, SW102

Commit message: update
Connections:
- net ESP32 Module/BOOT: now also SW101.2
- net ESP32 Module/RESET: now also SW102.2
- net GND: now also J101.4 (ID), J101.5 (GND), J101.6 (Shield), SW101.1, SW102.1
- net ESP32 Module/VCCUSB: now reaches J101.1 (VBUS)
- net ESP32 Module/D-: now reaches J101.2 (D-)
- net ESP32 Module/D+: now reaches J101.3 (D+)
Other:
- sheet ESP32 Module ports: added D+, D-, VCCUSB; removed none
- company: (none) -> CMOS-74A
- moved on the sheet: J101, SW101, SW102

Commit message: update
Other:
- sheet ESP32 Module ports: added CANH, CANL, PWM0, PWM1, PWM2, PWM3, PWM4, RX1, RX2, RXD0, SCK, SCL1, SCS, SDA1, SDI, SDO, TX1, TX2, TXD0; removed none
- sheet I2C_Peripherique ports: added PWM0, PWM1, PWM2, PWM3, PWM4, SCL0-E, SCL1-E, SCL2-E, SCL3-E, SDA0-E, SDA1-E, SDA2-E, SDA3-E; removed none

Commit message: update
Parts:
- SW101: footprint Button_Switch_THT:SW_Tactile_SKHH_Angled -> Button_Switch_SMD:SW_SPST_CK_RS282G05A3
Changed lines of the file:
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@@
 			)
 		)
-		(property "Footprint" "Button_Switch_THT:SW_Tactile_SKHH_Angled"
+		(property "Footprint" "Button_Switch_SMD:SW_SPST_CK_RS282G05A3"
 			(at 125.73 106.68 0)
 			(effects
@@
 			(at 125.73 106.68 0)
 			(effects
+				(font
+					(size 1.27 1.27)
+				)
+				(hide yes)
+			)
+		)
+		(property "UART" ""
+			(at 125.73 106.68 0)
+			(effects

Commit message: update
Connections:
- no-connect marks 1 -> 6
Other:
- sheet ESP32 Module ports: added E, IO8, RS, RW, T1CK, T2CK; removed none
- sheet I2C_Peripherique ports: added none; removed PWM0, PWM1, PWM2, PWM3, PWM4
