File: KICAD/CPU_ESP/V0.1/CPU/CPU.kicad_sch (KiCad schematic)
At the start: 4 parts, among them J101 USB_B_Mini, J102 Conn_01x04, SW101 SW_Push_45deg, SW102 SW_Push_45deg

Commit message: update
Other:
- added sheet SEVEN SEGMENTS (sevensegments.kicad_sch)
Changed lines of the file:
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@@
+	(wire
+		(pts
+			(xy 210.82 69.85) (xy 220.98 69.85)
+		)
+		(stroke
+			(width 0)
+			(type default)
+		)
+	)
 	(wire
 		(pts
@@
 		(pts
 			(xy 148.59 149.86) (xy 154.94 149.86)
+		)
+		(stroke
+			(width 0)
+			(type default)
+		)
+	)
+	(wire
+		(pts
+			(xy 210.82 72.39) (xy 220.98 72.39)
 		)
 		(stroke
@@
 		)
 	)
+	(label "SCL-5V"
+		(at 213.36 69.85 0)
+		(effects
+			(font
+				(size 1.27 1.27)
+			)
+			(justify left bottom)
+		)
+	)
 	(label "RESET"
 		(at 146.05 44.45 0)
@@
 	(label "PWM1"
 		(at 57.15 142.24 0)
+		(effects
+			(font
+				(size 1.27 1.27)
+			)
+			(justify left bottom)
+		)
+	)
+	(label "SDA-5V"
+		(at 213.36 72.39 0)
 		(effects
 			(font
@@
 				)
 			)
+		)
+	)
+	(sheet
+		(at 220.98 66.04)
+		(size 13.97 25.4)
+		(exclude_from_sim no)
+		(in_bom yes)
+		(on_board yes)
+		(dnp no)
+		(fields_autoplaced yes)
+		(stroke
+			(width 0.1524)
+			(type solid)
+		)
+		(fill
+			(color 0 0 0 0.0000)
+		)
+		(property "Sheetname" "SEVEN SEGMENTS"
+			(at 220.98 65.3284 0)
+			(effects
+				(font
+					(size 1.27 1.27)
+				)
+				(justify left bottom)
+			)
+		)
+		(property "Sheetfile" "sevensegments.kicad_sch"
+			(at 220.98 92.0246 0)
+			(effects
+				(font
+					(size 1.27 1.27)
+				)
+				(justify left top)
+			)
+		)
+		(pin "SCL-5V" input
+			(at 220.98 69.85 180)
+			(effects
+				(font
+					(size 1.27 1.27)
+				)
+				(justify left)
+			)
+		)
+		(pin "SDA-5V" input
+			(at 220.98 72.39 180)
+			(effects
+				(font
+					(size 1.27 1.27)
+				)
+				(justify left)
+			)
+		)
+		(instances
+			(project "CPU"
+				(path "/a676c576-12a0-418f-9fc1-1ecc8cb5a083"
+					(page "6")
+				)
+			)

Commit message: update
Other:
- sheet I2C_Peripherique ports: added none; removed SCL0, SCL2, SCL3, SDA0, SDA1, SDA2, SDA3
Changed lines of the file:
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@@
 	(wire
 		(pts
-			(xy 182.88 78.74) (xy 193.04 78.74)
-		)
-		(stroke
-			(width 0)
-			(type default)
-		)
-	)
-	(wire
-		(pts
 			(xy 92.71 115.57) (xy 102.87 115.57)
 		)
@@
 	(wire
 		(pts
-			(xy 182.88 73.66) (xy 193.04 73.66)
-		)
-		(stroke
-			(width 0)
-			(type default)
-		)
-	)
-	(wire
-		(pts
 			(xy 144.78 59.69) (xy 154.94 59.69)
 		)
@@
 	(wire
 		(pts
-			(xy 182.88 81.28) (xy 193.04 81.28)
-		)
-		(stroke
-			(width 0)
-			(type default)
-		)
-	)
-	(wire
-		(pts
 			(xy 92.71 152.4) (xy 102.87 152.4)
 		)
@@
 	(wire
 		(pts
-			(xy 182.88 83.82) (xy 193.04 83.82)
-		)
-		(stroke
-			(width 0)
-			(type default)
-		)
-	)
-	(wire
-		(pts
 			(xy 144.78 57.15) (xy 154.94 57.15)
 		)
@@
 	(wire
 		(pts
-			(xy 182.88 88.9) (xy 193.04 88.9)
-		)
-		(stroke
-			(width 0)
-			(type default)
-		)
-	)
-	(wire
-		(pts
 			(xy 227.33 31.75) (xy 234.95 31.75)
 		)
@@
 	(wire
 		(pts
-			(xy 182.88 86.36) (xy 193.04 86.36)
-		)
-		(stroke
-			(width 0)
-			(type default)
-		)
-	)
-	(wire
-		(pts
 			(xy 154.94 109.22) (xy 128.27 109.22)
 		)
@@
 	(wire
 		(pts
-			(xy 182.88 76.2) (xy 193.04 76.2)
-		)
-		(stroke
-			(width 0)
-			(type default)
-		)
-	)
-	(wire
-		(pts
 			(xy 182.88 67.31) (xy 193.04 67.31)
 		)
@@
 	(wire
 		(pts
-			(xy 182.88 71.12) (xy 193.04 71.12)
-		)
-		(stroke
-			(width 0)
-			(type default)
-		)
-	)
-	(wire
-		(pts
 			(xy 209.55 137.16) (xy 209.55 139.7)
 		)
@@
 		)
 	)
-	(label "IO1"
-		(at 184.15 73.66 0)
-		(effects
-			(font
-				(size 1.27 1.27)
-			)
-			(justify left bottom)
-		)
-	)
 	(label "D2"
 		(at 191.77 54.61 180)
@@
 		)
 	)
-	(label "IO3"
-		(at 184.15 78.74 0)
-		(effects
-			(font
-				(size 1.27 1.27)
-			)
-			(justify left bottom)
-		)
-	)
 	(label "SDA0-E"
 		(at 146.05 33.02 0)
@@
 		)
 	)
-	(label "IO7"
-		(at 184.15 88.9 0)
-		(effects
-			(font
-				(size 1.27 1.27)
-			)
-			(justify left bottom)
-		)
-	)
 	(label "SCL2-E"
 		(at 191.77 30.48 180)
@@
 		)
 	)
-	(label "IO5"
-		(at 184.15 83.82 0)
-		(effects
-			(font
-				(size 1.27 1.27)
-			)
-			(justify left bottom)
-		)
-	)
 	(label "D3"
 		(at 101.6 120.65 180)
@@
 		)
 	)
-	(label "IO4"
-		(at 184.15 81.28 0)
-		(effects
-			(font
-				(size 1.27 1.27)
-			)
-			(justify left bottom)
-		)
-	)
 	(label "IO2"
 		(at 146.05 54.61 0)
@@
 		)
 	)
-	(label "IO2"
-		(at 184.15 76.2 0)
+	(label "SDA1-E"
+		(at 55.88 161.29 0)
 		(effects
 			(font
@@
 		)
 	)
-	(label "IO0"
-		(at 184.15 71.12 0)
-		(effects
-			(font
-				(size 1.27 1.27)
-			)
-			(justify left bottom)
-		)
-	)
 	(label "SCL-5V"
 		(at 213.36 69.85 0)
@@
 		)
 	)
-	(label "IO6"
-		(at 184.15 86.36 0)
-		(effects
-			(font
-				(size 1.27 1.27)
-			)
-			(justify left bottom)
-		)
-	)
 	(label "PWM4"
 		(at 57.15 149.86 0)
@@
 		)
 	)
-	(label "SDA1"
-		(at 55.88 161.29 0)
-		(effects
-			(font
-				(size 1.27 1.27)
-			)
-			(justify left bottom)
-		)
-	)
 	(label "RW"
 		(at 101.6 135.89 180)
@@
 		)
 	)
-	(label "SCL1"
-		(at 55.88 158.75 0)
-		(effects
-			(font
-				(size 1.27 1.27)
-			)
-			(justify left bottom)
-		)
-	)
 	(label "RX2"
 		(at 148.59 135.89 0)
@@
 		)
 	)
+	(label "SCL1-E"
+		(at 55.88 158.75 0)
+		(effects
+			(font
+				(size 1.27 1.27)
+			)
+			(justify left bottom)
+		)
+	)
 	(label "RX1"
 		(at 97.79 170.18 0)
@@
 	(sheet
 		(at 154.94 19.05)
-		(size 27.94 73.66)
+		(size 27.94 52.578)
 		(exclude_from_sim no)
 		(in_bom yes)
@@
 		)
 		(property "Sheetfile" "I2C.kicad_sch"
-			(at 154.94 93.2946 0)
+			(at 154.94 72.2126 0)
 			(effects
 				(font
@@
 			)
 		)
-		(pin "SCL0" input
-			(at 154.94 30.48 180)
-			(effects
-				(font
-					(size 1.27 1.27)
-				)
-				(justify left)
-			)
-		)
 		(pin "SDA-5V" input
 			(at 182.88 25.4 0)
@@
 			)
 		)
-		(pin "SDA0" input
-			(at 154.94 33.02 180)
-			(effects
-				(font
-					(size 1.27 1.27)
-				)
-				(justify left)
-			)
-		)
 		(pin "D0" input
 			(at 182.88 49.53 0)
@@
 			)
 		)
-		(pin "SCL1" input
-			(at 154.94 36.83 180)
-			(effects
-				(font
-					(size 1.27 1.27)
-				)
-				(justify left)
-			)
-		)
-		(pin "SCL2" input
-			(at 182.88 30.48 0)
-			(effects
-				(font
-					(size 1.27 1.27)
-				)
-				(justify right)
-			)
-		)
-		(pin "SCL3" input
-			(at 182.88 36.83 0)
-			(effects
-				(font
-					(size 1.27 1.27)
-				)
-				(justify right)
-			)
-		)
 		(pin "SDA" input
 			(at 154.94 25.4 180)
@@
 			)
 		)
-		(pin "SDA1" input
-			(at 154.94 39.37 180)
+		(pin "RESET" input
+			(at 154.94 44.45 180)
 			(effects
 				(font
@@
 			)
 		)
-		(pin "SDA2" input
-			(at 182.88 33.02 0)
-			(effects
-				(font
-					(size 1.27 1.27)
-				)
-				(justify right)
-			)
-		)
-		(pin "SDA3" input
-			(at 182.88 39.37 0)
-			(effects
-				(font
-					(size 1.27 1.27)
-				)
-				(justify right)
-			)
-		)
-		(pin "RESET" input
-			(at 154.94 44.45 180)
+		(pin "SCL1-E" input
+			(at 154.94 36.83 180)
 			(effects
 				(font
@@
 			)
 		)
-		(pin "SCL0-E" input
-			(at 182.88 71.12 0)
+		(pin "SCL2-E" input
+			(at 182.88 30.48 0)
 			(effects
 				(font
@@
 			)
 		)
-		(pin "SCL1-E" input
-			(at 182.88 76.2 0)
+		(pin "SCL3-E" input
+			(at 182.88 36.83 0)
 			(effects
 				(font
@@
 			)
 		)
-		(pin "SCL2-E" input
-			(at 182.88 81.28 0)
+		(pin "SDA1-E" input
+			(at 154.94 39.37 180)
 			(effects
 				(font
 					(size 1.27 1.27)
 				)
-				(justify right)
+				(justify left)
 			)
 		)
-		(pin "SCL3-E" input
-			(at 182.88 86.36 0)
+		(pin "SDA2-E" input
+			(at 182.88 33.02 0)
 			(effects
 				(font
@@
 			)
 		)
-		(pin "SDA0-E" input
-			(at 182.88 73.66 0)
+		(pin "SDA3-E" input
+			(at 182.88 39.37 0)
 			(effects
 				(font
@@
 			)
 		)
-		(pin "SDA1-E" input
-			(at 182.88 78.74 0)
+		(pin "SDA0-E" input
+			(at 154.94 33.02 180)
 			(effects
 				(font
 					(size 1.27 1.27)
 				)
-				(justify right)
+				(justify left)
 			)
 		)
-		(pin "SDA2-E" input
-			(at 182.88 83.82 0)
+		(pin "SCL0-E" input
+			(at 154.94 30.48 180)
 			(effects
 				(font
 					(size 1.27 1.27)
 				)
-				(justify right)
+				(justify left)
 			)
 		)
-		(pin "SDA3-E" input
-			(at 182.88 88.9 0)
+		(pin "SCL1" input
+			(at 154.94 71.628 270)
 			(effects
 				(font
 					(size 1.27 1.27)
 				)
-				(justify right)
+				(justify left)
 			)
 		)

Commit message: PCB update
Connections:
- no-connect marks 6 -> 8
Other:
- sheet I2C_Peripherique ports: added SDA1; removed none
Changed lines of the file:
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@@
 	)
 	(no_connect
+		(at 102.87 167.64)
+	)
+	(no_connect
 		(at 102.87 180.34)
 	)
@@
 	)
 	(no_connect
+		(at 102.87 165.1)
+	)
+	(no_connect
 		(at 242.57 54.61)
 	)
@@
 	(wire
 		(pts
+			(xy 182.88 73.66) (xy 193.04 73.66)
+		)
+		(stroke
+			(width 0)
+			(type default)
+		)
+	)
+	(wire
+		(pts
 			(xy 92.71 135.89) (xy 102.87 135.89)
 		)
@@
 	(wire
 		(pts
+			(xy 182.88 71.12) (xy 193.04 71.12)
+		)
+		(stroke
+			(width 0)
+			(type default)
+		)
+	)
+	(wire
+		(pts
 			(xy 182.88 49.53) (xy 193.04 49.53)
 		)
@@
 		)
 	)
-	(label "TX0"
-		(at 97.79 167.64 0)
-		(effects
-			(font
-				(size 1.27 1.27)
-			)
-			(justify left bottom)
-		)
-	)
 	(label "SCL2-E"
 		(at 191.77 30.48 180)
@@
 		)
 	)
+	(label "SCL1"
+		(at 187.96 71.12 0)
+		(effects
+			(font
+				(size 1.27 1.27)
+			)
+			(justify left bottom)
+		)
+	)
 	(label "RS"
 		(at 101.6 138.43 180)
@@
 		)
 	)
+	(label "SDA1"
+		(at 187.96 73.66 0)
+		(effects
+			(font
+				(size 1.27 1.27)
+			)
+			(justify left bottom)
+		)
+	)
 	(label "TX1"
 		(at 148.59 133.35 0)
@@
 		)
 	)
-	(label "RX0"
-		(at 97.79 165.1 0)
-		(effects
-			(font
-				(size 1.27 1.27)
-			)
-			(justify left bottom)
-		)
-	)
 	(symbol
 		(lib_id "Connector_Generic:Conn_01x04")
@@
 	(sheet
 		(at 154.94 19.05)
-		(size 27.94 52.578)
+		(size 27.94 64.008)
 		(exclude_from_sim no)
 		(in_bom yes)
@@
 		)
 		(property "Sheetfile" "I2C.kicad_sch"
-			(at 154.94 72.2126 0)
+			(at 154.94 83.6426 0)
 			(effects
 				(font
@@
 		)
 		(pin "SCL1" input
-			(at 154.94 71.628 270)
+			(at 182.88 71.12 0)
 			(effects
 				(font
 					(size 1.27 1.27)
 				)
-				(justify left)
+				(justify right)
+			)
+		)
+		(pin "SDA1" input
+			(at 182.88 73.66 0)
+			(effects
+				(font
+					(size 1.27 1.27)
+				)
+				(justify right)
 			)
 		)

Commit message: PCB to control
Parts:
- J102: footprint Connector_Harwin:Harwin_M20-89004xx_1x04_P2.54mm_Horizontal -> Connector_JST:JST_GH_SM04B-GHS-TB_1x04-1MP_P1.25mm_Horizontal
Connections:
- net ESP32 Module/RESET is gone; now on net RESET: SW102.2
Changed lines of the file:
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@@
-	(wire
-		(pts
-			(xy 144.8539 44.4107) (xy 155.0139 44.4107)
-		)
-		(stroke
-			(width 0)
-			(type default)
-		)
-	)
 	(wire
 		(pts
@@
 		(pts
 			(xy 144.78 57.15) (xy 154.94 57.15)
+		)
+		(stroke
+			(width 0)
+			(type default)
+		)
+	)
+	(wire
+		(pts
+			(xy 144.78 44.45) (xy 154.94 44.45)
 		)
 		(stroke
@@
 		)
 	)
+	(label "IO0"
+		(at 146.05 49.53 0)
+		(effects
+			(font
+				(size 1.27 1.27)
+			)
+			(justify left bottom)
+		)
+	)
+	(label "SDI"
+		(at 148.59 152.4 0)
+		(effects
+			(font
+				(size 1.27 1.27)
+			)
+			(justify left bottom)
+		)
+	)
+	(label "PWM2"
+		(at 57.15 144.78 0)
+		(effects
+			(font
+				(size 1.27 1.27)
+			)
+			(justify left bottom)
+		)
+	)
+	(label "D6"
+		(at 191.77 64.77 180)
+		(effects
+			(font
+				(size 1.27 1.27)
+			)
+			(justify right bottom)
+		)
+	)
+	(label "T1CK"
+		(at 148.59 158.75 0)
+		(effects
+			(font
+				(size 1.27 1.27)
+			)
+			(justify left bottom)
+		)
+	)
+	(label "SCL1-E"
+		(at 146.05 36.83 0)
+		(effects
+			(font
+				(size 1.27 1.27)
+			)
+			(justify left bottom)
+		)
+	)
+	(label "TX0"
+		(at 148.59 128.27 0)
+		(effects
+			(font
+				(size 1.27 1.27)
+			)
+			(justify left bottom)
+		)
+	)
+	(label "IO0"
+		(at 57.15 113.03 0)
+		(effects
+			(font
+				(size 1.27 1.27)
+			)
+			(justify left bottom)
+		)
+	)
+	(label "PWM1"
+		(at 146.05 114.3 0)
+		(effects
+			(font
+				(size 1.27 1.27)
+			)
+			(justify left bottom)
+		)
+	)
+	(label "PWM3"
+		(at 57.15 147.32 0)
+		(effects
+			(font
+				(size 1.27 1.27)
+			)
+			(justify left bottom)
+		)
+	)
+	(label "RS"
+		(at 187.96 152.4 0)
+		(effects
+			(font
+				(size 1.27 1.27)
+			)
+			(justify left bottom)
+		)
+	)
+	(label "SCK"
+		(at 148.59 147.32 0)
+		(effects
+			(font
+				(size 1.27 1.27)
+			)
+			(justify left bottom)
+		)
+	)
+	(label "SCL1"
+		(at 187.96 71.12 0)
+		(effects
+			(font
+				(size 1.27 1.27)
+			)
+			(justify left bottom)
+		)
+	)
+	(label "RS"
+		(at 101.6 138.43 180)
+		(effects
+			(font
+				(size 1.27 1.27)
+			)
+			(justify right bottom)
+		)
+	)
+	(label "IO5"
+		(at 146.05 62.23 0)
+		(effects
+			(font
+				(size 1.27 1.27)
+			)
+			(justify left bottom)
+		)
+	)
+	(label "PWM4"
+		(at 57.15 149.86 0)
+		(effects
+			(font
+				(size 1.27 1.27)
+			)
+			(justify left bottom)
+		)
+	)
+	(label "PWM0"
+		(at 57.15 139.7 0)
+		(effects
+			(font
+				(size 1.27 1.27)
+			)
+			(justify left bottom)
+		)
+	)
+	(label "RESET"
+		(at 146.05 109.22 0)
+		(effects
+			(font
+				(size 1.27 1.27)
+			)
+			(justify left bottom)
+		)
+	)
 	(label "RESET"
 		(at 146.05 44.45 0)
-		(effects
-			(font
-				(size 1.27 1.27)
-			)
-			(justify left bottom)
-		)
-	)
-	(label "IO0"
-		(at 146.05 49.53 0)
-		(effects
-			(font
-				(size 1.27 1.27)
-			)
-			(justify left bottom)
-		)
-	)
-	(label "SDI"
-		(at 148.59 152.4 0)
-		(effects
-			(font
-				(size 1.27 1.27)
-			)
-			(justify left bottom)
-		)
-	)
-	(label "PWM2"
-		(at 57.15 144.78 0)
-		(effects
-			(font
-				(size 1.27 1.27)
-			)
-			(justify left bottom)
-		)
-	)
-	(label "D6"
-		(at 191.77 64.77 180)
-		(effects
-			(font
-				(size 1.27 1.27)
-			)
-			(justify right bottom)
-		)
-	)
-	(label "T1CK"
-		(at 148.59 158.75 0)
-		(effects
-			(font
-				(size 1.27 1.27)
-			)
-			(justify left bottom)
-		)
-	)
-	(label "SCL1-E"
-		(at 146.05 36.83 0)
-		(effects
-			(font
-				(size 1.27 1.27)
-			)
-			(justify left bottom)
-		)
-	)
-	(label "TX0"
-		(at 148.59 128.27 0)
-		(effects
-			(font
-				(size 1.27 1.27)
-			)
-			(justify left bottom)
-		)
-	)
-	(label "IO0"
-		(at 57.15 113.03 0)
-		(effects
-			(font
-				(size 1.27 1.27)
-			)
-			(justify left bottom)
-		)
-	)
-	(label "PWM1"
-		(at 146.05 114.3 0)
-		(effects
-			(font
-				(size 1.27 1.27)
-			)
-			(justify left bottom)
-		)
-	)
-	(label "PWM3"
-		(at 57.15 147.32 0)
-		(effects
-			(font
-				(size 1.27 1.27)
-			)
-			(justify left bottom)
-		)
-	)
-	(label "RS"
-		(at 187.96 152.4 0)
-		(effects
-			(font
-				(size 1.27 1.27)
-			)
-			(justify left bottom)
-		)
-	)
-	(label "SCK"
-		(at 148.59 147.32 0)
-		(effects
-			(font
-				(size 1.27 1.27)
-			)
-			(justify left bottom)
-		)
-	)
-	(label "SCL1"
-		(at 187.96 71.12 0)
-		(effects
-			(font
-				(size 1.27 1.27)
-			)
-			(justify left bottom)
-		)
-	)
-	(label "RS"
-		(at 101.6 138.43 180)
-		(effects
-			(font
-				(size 1.27 1.27)
-			)
-			(justify right bottom)
-		)
-	)
-	(label "IO5"
-		(at 146.05 62.23 0)
-		(effects
-			(font
-				(size 1.27 1.27)
-			)
-			(justify left bottom)
-		)
-	)
-	(label "PWM4"
-		(at 57.15 149.86 0)
-		(effects
-			(font
-				(size 1.27 1.27)
-			)
-			(justify left bottom)
-		)
-	)
-	(label "PWM0"
-		(at 57.15 139.7 0)
 		(effects
 			(font
@@
 			)
 		)
-		(property "Footprint" "Connector_Harwin:Harwin_M20-89004xx_1x04_P2.54mm_Horizontal"
+		(property "Footprint" "Connector_JST:JST_GH_SM04B-GHS-TB_1x04-1MP_P1.25mm_Horizontal"
 			(at 240.03 29.21 0)
 			(effects
@@
 			(at 240.03 29.21 0)
 			(effects
+				(font
+					(size 1.27 1.27)
+				)
+				(hide yes)
+			)
+		)
+		(property "UART" ""
+			(at 240.03 29.21 0)
+			(effects

Commit message: VSCODE update
Parts:
- added J103: Conn_01x04, Connector_JST:JST_GH_SM04B-GHS-TB_1x04-1MP_P1.25mm_Horizontal, symbol Connector_Generic:Conn_01x04
Connections:
- net +5VD: now also J103.2 (Pin_2)
- net GND: now also J103.1 (Pin_1)
- net RX1: now also J103.3 (Pin_3)
- net TX1: now also J103.4 (Pin_4)
Other:
- note added: "I2C EXTERNE"
- note added: "UART DEBUG"
- note added: "UART PROG/DEBUG"
