File: KICAD/CPU_ESP/V0.1/CPU/sevensegments.kicad_sch (KiCad schematic)
At the start: 7 parts, among them Q601 BSR19, Q602 BSR19, U601 SAA1064T

Commit message: update
Parts:
- U601: footprint Package_SO:SO-24_5.3x15mm_P1.27mm -> Package_SO:SOP-24_7.5x15.4mm_P1.27mm
Changed lines of the file:
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@@
 			)
 		)
-		(property "Footprint" "Package_SO:SO-24_5.3x15mm_P1.27mm"
+		(property "Footprint" "Package_SO:SOP-24_7.5x15.4mm_P1.27mm"
 			(at 90.805 92.075 0)
 			(effects
@@
 			)
 		)
+		(property "UART" ""
+			(at 137.16 93.98 0)
+			(effects
+				(font
+					(size 1.27 1.27)
+				)
+				(hide yes)
+			)
+		)
