File: KICAD/CPU_ESP/V0.1/CPU/CPU.kicad_pcb (KiCad board)
At the start: 2 copper layers, 100 x 100 mm, 18 parts, among them J101 USB_B_Mini, J501 Conn_02x20_Odd_Even, J502 Conn_02x20_Odd_Even, SW101 SW_Push_45deg, SW102 SW_Push_45deg, U301 LM1117DT-2.5, U401 ESP32-WROOM-32

Commit message: Update
Parts:
- added D201: D_Schottky, Diode_SMD:D_1206_3216Metric, F.Cu at (220.6, 129.5)
- added R201: 150, Resistor_SMD:R_0603_1608Metric, F.Cu at (207.7, 129.1)
- added R202: 330, Resistor_SMD:R_0603_1608Metric, F.Cu at (207.7, 131.6)
- added R203: 2.2K, Resistor_SMD:R_0603_1608Metric, F.Cu at (207.7, 134.1)
- added R204: 2.2K, Resistor_SMD:R_0603_1608Metric, F.Cu at (207.7, 136.6)
- added R205: 2.2K, Resistor_SMD:R_0603_1608Metric, F.Cu at (150.0, 128.7)
- added R206: 2.2K, Resistor_SMD:R_0603_1608Metric, F.Cu at (165.5, 120.7)
- added R207: NC, Resistor_SMD:R_0603_1608Metric, F.Cu at (204.5, 134.7)
- added R208: 0, Resistor_SMD:R_0603_1608Metric, F.Cu at (211.7, 129.1)
- added R209: NC, Resistor_SMD:R_0603_1608Metric, F.Cu at (211.7, 131.6)
- added R210: 0, Resistor_SMD:R_0603_1608Metric, F.Cu at (211.7, 134.1)
- added R211: NC, Resistor_SMD:R_0603_1608Metric, F.Cu at (211.7, 136.6)
- added R212: 0, Resistor_SMD:R_0603_1608Metric, F.Cu at (204.5, 140.2)
- added R213: NC, Resistor_SMD:R_0603_1608Metric, F.Cu at (155.0, 130.7)
- added R214: 0, Resistor_SMD:R_0603_1608Metric, F.Cu at (155.0, 134.2)
- added R215: NC, Resistor_SMD:R_0603_1608Metric, F.Cu at (215.8, 129.1)
- added R216: 0, Resistor_SMD:R_0603_1608Metric, F.Cu at (215.8, 131.6)
- added R217: NC, Resistor_SMD:R_0603_1608Metric, F.Cu at (215.8, 134.1)
- added R218: 0, Resistor_SMD:R_0603_1608Metric, F.Cu at (215.8, 136.6)
- added U201: PCF8563T, Package_SO:SOIC-8_3.9x4.9mm_P1.27mm, F.Cu at (139.0, 133.1)
- added U204: TCA9544A, Package_SO:TSSOP-20_4.4x6.5mm_P0.65mm, F.Cu at (164.9, 136.1)
- added U205: MCP23017_SO, Package_SO:SOIC-28W_7.5x17.9mm_P1.27mm, F.Cu at (197.3, 130.7)
- added U206: AT24CS01-MAHM, Package_DFN_QFN:DFN-8-1EP_3x2mm_P0.5mm_EP1.3x1.5mm, F.Cu at (159.4, 121.2)

Commit message: Update
Parts:
- added C201: C, Capacitor_SMD:C_0603_1608Metric, F.Cu at (103.7, 112.4)
- added C202: 10F/2.7V, Capacitor_THT:CP_Radial_Tantal_D5.0mm_P5.00mm, F.Cu at (94.9, 102.7)
- added C203: 10F/2.7V, Capacitor_THT:CP_Radial_Tantal_D5.0mm_P5.00mm, F.Cu at (94.9, 111.2)
- added D202: RED, LED_SMD:LED_0603_1608Metric, F.Cu at (103.7, 109.8)
- added J102: Conn_01x04, Connector_Harwin:Harwin_M20-89004xx_1x04_P2.54mm_Horizontal, F.Cu at (210.0, 154.5)
- added R105: 2.2k, Resistor_SMD:R_0603_1608Metric, F.Cu at (176.2, 121.4)
- added R106: 2.2k, Resistor_SMD:R_0603_1608Metric, F.Cu at (176.2, 123.9)
- added R109: 2.2k, Resistor_SMD:R_0603_1608Metric, F.Cu at (176.2, 126.5)
- added R110: 2.2k, Resistor_SMD:R_0603_1608Metric, F.Cu at (176.2, 129.0)
- added R111: 2.2k, Resistor_SMD:R_0603_1608Metric, F.Cu at (176.2, 131.5)
- added R112: 2.2k, Resistor_SMD:R_0603_1608Metric, F.Cu at (176.2, 134.0)
- added R113: 2.2k, Resistor_SMD:R_0603_1608Metric, F.Cu at (176.2, 136.5)
- added R114: 2.2k, Resistor_SMD:R_0603_1608Metric, F.Cu at (176.2, 139.0)
- added U202: LM75A, Package_SO:SOIC-8_3.9x4.9mm_P1.27mm, F.Cu at (105.9, 101.8)
- added U203: PCA9306, Package_SO:VSSOP-8_2.3x2mm_P0.5mm, F.Cu at (104.9, 106.8)
- added Y201: 32.768Khz, Crystal:Crystal_SMD_TXC_9HT11-2Pin_2.0x1.2mm, F.Cu at (107.6, 110.0)
Connections:
- net /CMOS_BUS/E renamed /E
- net /CMOS_BUS/IO0 renamed /IO0
- net /CMOS_BUS/IO1 renamed /IO1
- net /CMOS_BUS/IO2 renamed /IO2
- net /CMOS_BUS/IO3 renamed /IO3
- net /CMOS_BUS/IO4 renamed /IO4
- net /CMOS_BUS/IO5 renamed /IO5
- net /CMOS_BUS/IO6 renamed /IO6
- net /CMOS_BUS/IO7 renamed /IO7
- net /CMOS_BUS/IO8 renamed /IO8
- net /CMOS_BUS/IO9 renamed /IO9
- net /CMOS_BUS/RETRO renamed /RETRO
- net /CMOS_BUS/RS renamed /RS
- net /CMOS_BUS/RST renamed /RESET
- net /CMOS_BUS/RW renamed /RW
- net /I2C_Peripherique/RST renamed /I2C_Peripherique/RESET
- J502 pad 12: /CMOS_BUS/D0 -> /D0
- J502 pad 13: /CMOS_BUS/D1 -> /D1
- J502 pad 14: /CMOS_BUS/D2 -> /D2
- J502 pad 15: /CMOS_BUS/D3 -> /D3
- J502 pad 16: /CMOS_BUS/D4 -> /D4
- J502 pad 17: /CMOS_BUS/D5 -> /D5
- J502 pad 18: /CMOS_BUS/D6 -> /D6
- J502 pad 19: /CMOS_BUS/D7 -> /D7
- U205 pad 1: /I2C_Peripherique/D0 -> /D0
- U205 pad 2: /I2C_Peripherique/D1 -> /D1
- U205 pad 3: /I2C_Peripherique/D2 -> /D2
- U205 pad 4: /I2C_Peripherique/D3 -> /D3
- U205 pad 5: /I2C_Peripherique/D4 -> /D4
- U205 pad 6: /I2C_Peripherique/D5 -> /D5
- U205 pad 7: /I2C_Peripherique/D6 -> /D6
- U205 pad 8: /I2C_Peripherique/D7 -> /D7
- U401 pad 33: unconnected-(U401-IO21-Pad33) -> /ESP32 Module/SDA
- U401 pad 34: unconnected-(U401-RXD0/IO3-Pad34) -> /ESP32 Module/RX0
- U401 pad 35: unconnected-(U401-TXD0/IO1-Pad35) -> /ESP32 Module/TX0
- U401 pad 36: unconnected-(U401-IO22-Pad36) -> /ESP32 Module/SCL

Commit message: update
Parts:
- added C405: 100n, Capacitor_SMD:C_0603_1608Metric, F.Cu at (230.8, 105.4)
- added C406: 100n, Capacitor_SMD:C_0603_1608Metric, F.Cu at (230.8, 107.9)
- added C407: 4.7µ/10V, Capacitor_Tantalum_SMD:CP_EIA-3216-12_Kemet-S, F.Cu at (244.1, 117.8)
- added C408: 100n, Capacitor_SMD:C_0603_1608Metric, F.Cu at (230.8, 110.4)
- added D403: LED_Dual_KAK, LED_SMD:LED_Kingbright_KPA-3010_3x2x1mm, F.Cu at (162.5, 153.5)
- added D404: LED_Dual_KAK, LED_SMD:LED_Kingbright_KPA-3010_3x2x1mm, F.Cu at (169.5, 153.5)
- added R402: 2k2, Resistor_SMD:R_0603_1608Metric, F.Cu at (230.8, 112.9)
- added R403: 2k2, Resistor_SMD:R_0603_1608Metric, F.Cu at (230.8, 115.4)
- added R405: NC, Resistor_SMD:R_0603_1608Metric, F.Cu at (230.8, 118.0)
- added R408: 4k7, Resistor_SMD:R_0603_1608Metric, F.Cu at (230.8, 120.5)
- added R409: 4k7, Resistor_SMD:R_0603_1608Metric, F.Cu at (230.8, 123.0)
- added R410: 120, Resistor_SMD:R_1206_3216Metric, F.Cu at (244.0, 121.0)
- added R411: 330, Resistor_SMD:R_0603_1608Metric, F.Cu at (162.2, 148.5)
- added R412: 330, Resistor_SMD:R_0603_1608Metric, F.Cu at (164.2, 148.5)
- added R413: 330, Resistor_SMD:R_0603_1608Metric, F.Cu at (169.2, 148.5)
- added R414: 330, Resistor_SMD:R_0603_1608Metric, F.Cu at (171.2, 148.5)
- added U402: FT232RL, Package_SO:SSOP-28_5.3x10.2mm_P0.65mm, F.Cu at (238.1, 110.2)
- added U403: TJA1051T, Package_SO:SOIC-8_3.9x4.9mm_P1.27mm, F.Cu at (237.0, 119.5)
- C201: renamed from C202; footprint Capacitor_THT:CP_Radial_Tantal_D5.0mm_P5.00mm -> Capacitor_THT:CP_Radial_Tantal_D10.5mm_P5.00mm
- C202: renamed from C203; footprint Capacitor_THT:CP_Radial_Tantal_D5.0mm_P5.00mm -> Capacitor_THT:CP_Radial_Tantal_D10.5mm_P5.00mm
- C203: renamed from C201; value C -> 10n
- SW101: footprint Button_Switch_THT:SW_Tactile_SKHH_Angled -> Button_Switch_SMD:SW_SPST_CK_RS282G05A3
- U206: footprint Package_DFN_QFN:DFN-8-1EP_3x2mm_P0.5mm_EP1.3x1.5mm -> Package_SO:SOIC-8_5.3x5.3mm_P1.27mm
- Y201: value 32.768Khz -> 32.278kHz; footprint Crystal:Crystal_SMD_TXC_9HT11-2Pin_2.0x1.2mm -> Crystal:Crystal_SMD_Abracon_ABS25-4Pin_8.0x3.8mm
- moved C202 73.7 mm to (165.0, 134.0), turned to -90 degrees
- moved C201 72.5 mm to (165.0, 121.5), turned to -90 degrees
- moved U201 70.8 mm to (176.5, 107.0)
- moved D201 55.4 mm to (168.0, 112.0), turned to 90 degrees
- moved R206 48.2 mm to (121.0, 139.2)
- moved C203 47.8 mm to (151.2, 117.0)
- moved U301 45.7 mm to (149.6, 84.7), turned to 90 degrees
- moved R201 44.5 mm to (165.0, 116.7), turned to -90 degrees
- moved U204 42.3 mm to (196.5, 108.0)
- moved Y201 40.3 mm to (147.8, 112.4), turned to -90 degrees
- moved C404 34.8 mm to (188.0, 94.7), turned to -90 degrees
- moved R401 31.4 mm to (161.8, 80.3), turned to 90 degrees
- moved C403 29.3 mm to (158.5, 77.0), turned to 180 degrees
- moved R213 27.4 mm to (129.0, 139.3)
- moved C304 26.7 mm to (147.5, 95.5), turned to 180 degrees
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- renumbered R204 to R202, R202 to R204, R208 to R207, U202 to U201, U203 to U202, U201 to U203
Connections:
- net /CMOS_BUS/SCL0 renamed /SCL0-E
- net /CMOS_BUS/SCL2 renamed /SCL2-E
- net /CMOS_BUS/SDA0 renamed /SDA0-E
- net /CMOS_BUS/SDA2 renamed /SDA2-E
- net /ESP32 Module/RX0 renamed /ESP32 Module/RXD0
- net /ESP32 Module/TX0 renamed /ESP32 Module/TXD0
- C203 pad 1: Net-(U201-OSCO) -> Net-(U203-OSCO)
- J101 pad 1: unconnected-(J101-VBUS-Pad1) -> /ESP32 Module/VCCUSB
- J101 pad 2: unconnected-(J101-D--Pad2) -> /ESP32 Module/D-
- J101 pad 3: unconnected-(J101-D+-Pad3) -> /ESP32 Module/D+
- J101 pad 4: unconnected-(J101-ID-Pad4) -> GND
- J101 pad 5: unconnected-(J101-GND-Pad5) -> GND
- J101 pad 6: unconnected-(J101-Shield-Pad6) -> GND
- J102 pad 4: /SCL-5V -> /SDA-5V
- J501 pad 23: /CMOS_BUS/PWM0 -> /PWM0
- J501 pad 24: /CMOS_BUS/PWM1 -> /PWM1
- J501 pad 25: /CMOS_BUS/PWM2 -> /PWM2
- J501 pad 26: /CMOS_BUS/PWM3 -> /PWM3
- J501 pad 27: /CMOS_BUS/PWM4 -> /PWM4
- J502 pad 10: /CMOS_BUS/SDO -> /SDO
- J502 pad 33: /CMOS_BUS/SDA1 -> /SDA1-E
- J502 pad 34: /CMOS_BUS/SCL1 -> /SCL1-E
- J502 pad 7: /CMOS_BUS/SCK -> /SCK
- J502 pad 8: /CMOS_BUS/SDI -> /SDI
- J502 pad 9: /CMOS_BUS/SCS -> /SCS
- R105 pad 2: /I2C_Peripherique/SCL2 -> /IO4
- R106 pad 2: /I2C_Peripherique/SCL2 -> /IO4
- R109 pad 2: /I2C_Peripherique/SCL1 -> /IO2
- R110 pad 2: /I2C_Peripherique/SDA1 -> /IO3
- R111 pad 2: /I2C_Peripherique/SCL0 -> /IO0
- R112 pad 2: /I2C_Peripherique/SDA0 -> /IO1
- R113 pad 2: /I2C_Peripherique/SCL3 -> /IO6
- R114 pad 2: /I2C_Peripherique/SDA3 -> /IO7
- R202 pad 2: /I2C_Peripherique/SDA -> /SDA
- R203 pad 2: /I2C_Peripherique/SCL -> /SCL
- R206 pad 2: /SCL-5V -> /SDA-5V
- SW101 pad 1: unconnected-(SW101-Pad1) -> GND
- SW101 pad 2: unconnected-(SW101-Pad2) -> /ESP32 Module/BOOT
- SW102 pad 1: unconnected-(SW102-Pad1) -> GND
- SW102 pad 2: unconnected-(SW102-Pad2) -> /ESP32 Module/RESET
- U201 pad 1: /SCL-5V -> /SDA-5V
- U202 pad 3: /I2C_Peripherique/SCL -> /SCL
- U202 pad 4: /I2C_Peripherique/SDA -> /SDA
- U202 pad 5: /SCL-5V -> /SDA-5V
- U203 pad 1: Net-(U201-OSCI) -> Net-(U203-OSCI)
- U203 pad 2: Net-(U201-OSCO) -> Net-(U203-OSCO)
- U203 pad 5: /SCL-5V -> /SDA-5V
- U204 pad 12: /I2C_Peripherique/SDA2 -> /IO5
- U204 pad 13: /I2C_Peripherique/SCL2 -> /IO4
- U204 pad 15: /I2C_Peripherique/SDA3 -> /IO7
- U204 pad 16: /I2C_Peripherique/SCL3 -> /IO6
- U204 pad 18: /I2C_Peripherique/SCL -> /SCL1-E
- U204 pad 19: /I2C_Peripherique/SDA -> /SDA1-E
- U204 pad 5: /I2C_Peripherique/SDA0 -> /IO1
- U204 pad 6: /I2C_Peripherique/SCL0 -> /IO0
- U204 pad 8: /I2C_Peripherique/SDA1 -> /IO3
- U204 pad 9: /I2C_Peripherique/SCL1 -> /IO2
- U205 pad 12: /I2C_Peripherique/SDA -> /SCL
- U205 pad 13: /I2C_Peripherique/SCL -> /SDA
- U205 pad 21: /I2C_Peripherique/IO0 -> /IO0
- U205 pad 22: /I2C_Peripherique/IO1 -> /IO1
- U205 pad 23: /I2C_Peripherique/IO2 -> /IO2
- U205 pad 24: /I2C_Peripherique/IO3 -> /IO3
- U205 pad 25: /I2C_Peripherique/IO4 -> /IO4
- U205 pad 26: /I2C_Peripherique/IO5 -> /IO5
- U205 pad 27: /I2C_Peripherique/IO6 -> /IO6
- U205 pad 28: /I2C_Peripherique/IO7 -> /IO7
- U206 pad 5: /SCL-5V -> /SDA-5V
- U401 pad 10: unconnected-(U401-IO25-Pad10) -> /PWM2
- U401 pad 11: unconnected-(U401-IO26-Pad11) -> /PWM3
- U401 pad 12: unconnected-(U401-IO27-Pad12) -> /PWM4
- U401 pad 14: unconnected-(U401-IO12-Pad14) -> Net-(U401-IO12)
- U401 pad 19: unconnected-(U401-SCS/CMD-Pad19) -> /SCS
- U401 pad 20: unconnected-(U401-SCK/CLK-Pad20) -> /SCK
- U401 pad 21: unconnected-(U401-SDO/SD0-Pad21) -> /SDO
- U401 pad 22: unconnected-(U401-SDI/SD1-Pad22) -> /SDI
- U401 pad 24: unconnected-(U401-IO2-Pad24) -> Net-(U401-IO2)
- U401 pad 26: unconnected-(U401-IO4-Pad26) -> Net-(U401-IO4)
- U401 pad 27: unconnected-(U401-IO16-Pad27) -> /RX1
- U401 pad 28: unconnected-(U401-IO17-Pad28) -> /TX1
- U401 pad 29: unconnected-(U401-IO5-Pad29) -> Net-(U401-IO5)
- U401 pad 30: unconnected-(U401-IO18-Pad30) -> /SDA1
- U401 pad 31: unconnected-(U401-IO19-Pad31) -> /SCL1
- U401 pad 33: /ESP32 Module/SDA -> /SDA
- U401 pad 36: /ESP32 Module/SCL -> /SCL
- U401 pad 4: unconnected-(U401-SENSOR_VP-Pad4) -> /ESP32 Module/CAN-TX
- U401 pad 5: unconnected-(U401-SENSOR_VN-Pad5) -> /ESP32 Module/CAN-RX
- U401 pad 6: unconnected-(U401-IO34-Pad6) -> /RX2
- U401 pad 7: unconnected-(U401-IO35-Pad7) -> /TX2
- U401 pad 8: unconnected-(U401-IO32-Pad8) -> /PWM0
- U401 pad 9: unconnected-(U401-IO33-Pad9) -> /PWM1
- Y201 pad 1: Net-(U201-OSCO) -> Net-(U203-OSCI)
- Y201 pad 2: Net-(U201-OSCI) -> unconnected-(Y201-Pad2)
Routing:
- net GND: track 0.00 -> 74.3 mm
- net +3.3V: track 0.00 -> 50.8 mm, vias 0 -> 4
- net /SDA-5V: track 0.00 -> 34.6 mm, vias 0 -> 3
- net /SCL-5V: track 0.00 -> 25.6 mm
- net +5VD: track 0.00 -> 11.3 mm, vias 0 -> 2
- net Net-(D201-K): track 0.00 -> 10.00 mm
- net Net-(U203-OSCO): track 0.00 -> 8.20 mm
- net Net-(C201-Pad2): track 0.00 -> 7.50 mm
- net /ESP32 Module/RESET: track 0.00 -> 7.00 mm
- net Net-(U203-OSCI): track 0.00 -> 5.98 mm
- net /ESP32 Module/BOOT: track 0.00 -> 4.62 mm
- net Net-(C201-Pad1): track 0.00 -> 4.00 mm
- net Net-(D404-K1): track 0.00 -> 3.68 mm
- net Net-(D403-K1): track 0.00 -> 3.68 mm
- net Net-(D404-K2): track 0.00 -> 3.13 mm
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
Commit message: update
Parts:
- removed the R207 at (204.5, 134.7)
- removed R209, R211, R213, R215, R217: NC, Resistor_SMD:R_0603_1608Metric
- removed U206: AT24CS01-MAHM, Package_SO:SOIC-8_5.3x5.3mm_P1.27mm
- added C601: 100n, Capacitor_SMD:C_0603_1608Metric, F.Cu at (252.2, 146.0)
- added C602: 2.7n, Capacitor_SMD:C_0603_1608Metric, F.Cu at (252.2, 148.5)
- added D401: ORANGE, LED_SMD:LED_0603_1608Metric, F.Cu at (255.5, 112.2)
- added D402: ORANGE, LED_SMD:LED_0603_1608Metric, F.Cu at (255.5, 114.8)
- added J601: ~, Connector_PinSocket_2.54mm:PinSocket_2x05_P2.54mm_Horizontal, F.Cu at (189.5, 141.4)
- added J602: ~, Connector_PinSocket_2.54mm:PinSocket_2x05_P2.54mm_Horizontal, F.Cu at (204.7, 141.5)
- added L401: 22µ, Inductor_SMD:L_1008_2520Metric, F.Cu at (255.9, 118.0)
- added Q601: BSR19, Package_TO_SOT_SMD:SOT-23, F.Cu at (247.8, 147.1)
- added Q602: BSR19, Package_TO_SOT_SMD:SOT-23, F.Cu at (247.8, 151.8)
- added R404: 0, Resistor_SMD:R_0603_1608Metric, F.Cu at (251.4, 112.2)
- added R406: 0, Resistor_SMD:R_0603_1608Metric, F.Cu at (251.4, 114.7)
- added R407: 0, Resistor_SMD:R_0603_1608Metric, F.Cu at (251.4, 117.2)
- added U207: AT24CS01-SSHM, Package_SO:SOIC-8_5.3x5.3mm_P1.27mm, F.Cu at (159.0, 106.5)
- added U601: SAA1064T, Package_SO:SO-24_5.3x15mm_P1.27mm, F.Cu at (250.6, 136.5)
- moved J102 70.0 mm to (277.5, 155.0)
- moved J502 6.92 mm to (217.5, 62.0)
- moved J501 6.20 mm to (135.0, 62.0)
- moved R212 2.33 mm to (204.7, 137.9)
Connections:
- J502 pad 23: /CMOS_BUS/UART-RX0 -> /RX0
- J502 pad 24: /CMOS_BUS/UART-TX0 -> /TX0
- J502 pad 25: /CMOS_BUS/UART-RX1 -> /RX1
- J502 pad 26: /CMOS_BUS/UART-TX1 -> /TX1
- J502 pad 27: /CMOS_BUS/UART-RX2 -> /RX2
- J502 pad 28: /CMOS_BUS/UART-TX2 -> /TX2
- J502 pad 3: /CMOS_BUS/T1CK -> /T1CK
- J502 pad 33: /SDA1-E -> /SDA1
- J502 pad 34: /SCL1-E -> /SCL1
- J502 pad 4: /CMOS_BUS/T2CK -> /T2CK
- J502 pad 5: /CMOS_BUS/CANRX -> /CANH
- J502 pad 6: /CMOS_BUS/CANTX -> /CANL
- R410 pad 1: /ESP32 Module/CANL -> /CANL
- R410 pad 2: /ESP32 Module/CANH -> /CANH
- U401 pad 13: unconnected-(U401-IO14-Pad13) -> /RW
- U401 pad 16: unconnected-(U401-IO13-Pad16) -> /E
- U401 pad 17: unconnected-(U401-SHD/SD2-Pad17) -> /T1CK
- U401 pad 18: unconnected-(U401-SWP/SD3-Pad18) -> /T2CK
- U401 pad 23: unconnected-(U401-IO15-Pad23) -> /RS
- U401 pad 34: /ESP32 Module/RXD0 -> /RX0
- U401 pad 35: /ESP32 Module/TXD0 -> /TX0
- U401 pad 37: unconnected-(U401-IO23-Pad37) -> /IO8
- U403 pad 6: /ESP32 Module/CANL -> /CANL
- U403 pad 7: /ESP32 Module/CANH -> /CANH

Commit message: update
Parts:
- removed R105, R106, R109, R110, R111, R112, R113, R114: 2.2k, Resistor_SMD:R_0603_1608Metric
- added R208: 2k2, Resistor_SMD:R_0603_1608Metric_Pad0.98x0.95mm_HandSolder, F.Cu at (204.5, 96.6)
- added R209: 2k2, Resistor_SMD:R_0603_1608Metric_Pad0.98x0.95mm_HandSolder, F.Cu at (206.0, 96.6)
- added R211: 2k2, Resistor_SMD:R_0603_1608Metric_Pad0.98x0.95mm_HandSolder, F.Cu at (207.5, 96.6)
- added R213: 2k2, Resistor_SMD:R_0603_1608Metric_Pad0.98x0.95mm_HandSolder, F.Cu at (209.0, 96.6)
- added R215: 2k2, Resistor_SMD:R_0603_1608Metric_Pad0.98x0.95mm_HandSolder, F.Cu at (208.5, 108.0)
- added R217: 2k2, Resistor_SMD:R_0603_1608Metric_Pad0.98x0.95mm_HandSolder, F.Cu at (210.1, 108.0)
- U601: footprint Package_SO:SO-24_5.3x15mm_P1.27mm -> Package_SO:SOP-24_7.5x15.4mm_P1.27mm
- moved U202 99.8 mm to (200.7, 78.7)
- moved R214 74.0 mm to (193.5, 98.0), turned to 180 degrees
- moved R212 73.4 mm to (278.1, 134.6), turned to 0 degrees
- moved U205 72.1 mm to (269.3, 125.9)
- moved R207 66.4 mm to (278.1, 131.6)
- moved R210 66.3 mm to (278.1, 133.1)
- moved D202 63.7 mm to (167.4, 107.7), turned to 180 degrees
- moved C602 63.6 mm to (194.1, 122.7), turned to 90 degrees
- moved Q602 61.7 mm to (188.2, 135.6)
- moved R202 57.9 mm to (195.3, 80.0)
- moved R203 50.5 mm to (197.9, 84.6)
- moved U601 48.8 mm to (202.3, 129.2)
- moved R204 43.9 mm to (170.9, 107.7)
- moved R218 41.9 mm to (193.5, 101.1), turned to 180 degrees
- moved R216 39.0 mm to (193.5, 99.6), turned to 180 degrees
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Connections:
- J502 pad 33: /SDA1 -> /SDA1-E
- J502 pad 34: /SCL1 -> /SCL1-E
- U204 pad 12: /IO5 -> /SDA2-E
- U204 pad 13: /IO4 -> /SCL2-E
- U204 pad 15: /IO7 -> unconnected-(U204-SD3-Pad15)
- U204 pad 16: /IO6 -> unconnected-(U204-SC3-Pad16)
- U204 pad 18: /SCL1-E -> /I2C_Peripherique/SCL1
- U204 pad 19: /SDA1-E -> /I2C_Peripherique/SDA1
- U204 pad 5: /IO1 -> /SDA0-E
- U204 pad 6: /IO0 -> /SCL0-E
- U204 pad 8: /IO3 -> /SDA1-E
- U204 pad 9: /IO2 -> /SCL1-E
Routing:
- net /SDA1-E: track 0.00 -> 32.0 mm, vias 0 -> 4
- net /SCL1-E: track 0.00 -> 29.5 mm, vias 0 -> 4
- net Net-(J602-Pin_2): track 0.00 -> 27.6 mm, vias 0 -> 2
- net /SEVEN SEGMENTS/P34: track 0.00 -> 26.7 mm, vias 0 -> 2
- net /SEVEN SEGMENTS/G34: track 0.00 -> 24.6 mm, vias 0 -> 1
- net /SDA0-E: track 0.00 -> 24.2 mm, vias 0 -> 2
- net /SCL0-E: track 0.00 -> 22.7 mm, vias 0 -> 2
- net /SEVEN SEGMENTS/F34: track 0.00 -> 22.5 mm
- net Net-(J602-Pin_1): track 0.00 -> 22.5 mm
- net Net-(J602-Pin_8): track 0.00 -> 22.2 mm, vias 0 -> 1
- net Net-(J602-Pin_4): track 0.00 -> 21.5 mm
- net /SEVEN SEGMENTS/D34: track 0.00 -> 20.2 mm, vias 0 -> 1
- net /SEVEN SEGMENTS/E34: track 0.00 -> 19.1 mm
- net /SEVEN SEGMENTS/C34: track 0.00 -> 18.5 mm
- net Net-(J602-Pin_6): track 0.00 -> 17.8 mm
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
Commit message: PCB update
Parts:
- added R219: 2k2, Resistor_SMD:R_0603_1608Metric, F.Cu at (202.2, 95.6)
- added R220: 2k2, Resistor_SMD:R_0603_1608Metric, F.Cu at (200.7, 95.6)
- moved R212 146.1 mm to (141.0, 84.1), turned to 180 degrees
- moved R210 145.0 mm to (141.0, 85.6), turned to 180 degrees
- moved R207 144.1 mm to (141.0, 87.1), turned to 180 degrees
- moved D401 129.4 mm to (129.3, 140.9), turned to -90 degrees
- moved D402 127.3 mm to (129.3, 131.1), turned to 90 degrees
- moved L401 125.6 mm to (132.6, 142.0), turned to 180 degrees
- moved U205 123.4 mm to (150.4, 92.8), turned to 180 degrees
- moved R404 105.5 mm to (149.0, 137.4)
- moved R407 105.0 mm to (149.0, 140.4)
- moved R406 104.6 mm to (149.0, 135.9)
- moved R408 103.0 mm to (129.3, 137.7), turned to -90 degrees
- moved R409 102.1 mm to (129.3, 134.3), turned to 90 degrees
- moved R403 101.7 mm to (131.6, 137.7), turned to 90 degrees
- moved R402 101.5 mm to (131.6, 134.4), turned to 90 degrees
- moved U402 101.1 mm to (140.3, 135.6), turned to 180 degrees
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Connections:
- J502 pad 23: /RX0 -> /CMOS_BUS/UART-RX0
- J502 pad 24: /TX0 -> /CMOS_BUS/UART-TX0
- U204 pad 18: /I2C_Peripherique/SCL1 -> /SCL1
- U204 pad 19: /I2C_Peripherique/SDA1 -> /SDA1
Routing:
- net GND: track 90.5 -> 261.7 mm
- net /RX0: track 0.00 -> 97.7 mm, vias 0 -> 2
- net /TX0: track 0.00 -> 95.7 mm, vias 0 -> 2
- net /ESP32 Module/RESET: track 7.00 -> 82.9 mm, vias 0 -> 3
- net /ESP32 Module/CAN-RX: track 0.00 -> 68.7 mm, vias 0 -> 2
- net +5VD: track 23.5 -> 91.8 mm, vias 4 -> 9
- net /IO8: track 0.00 -> 66.2 mm, vias 0 -> 1
- net /SCL: track 0.00 -> 60.2 mm, vias 0 -> 5
- net /SDA: track 0.00 -> 53.6 mm, vias 0 -> 4
- net /ESP32 Module/CAN-TX: track 0.00 -> 50.6 mm, vias 0 -> 2
- net /SCL1: track 0.00 -> 41.1 mm, vias 0 -> 4
- net /PWM1: track 0.00 -> 36.2 mm, vias 0 -> 1
- net /PWM3: track 0.00 -> 35.6 mm, vias 0 -> 1
- net /SDA1: track 0.00 -> 34.5 mm, vias 0 -> 4
- net /PWM0: track 0.00 -> 33.8 mm, vias 0 -> 1
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
Commit message: PCB update
Parts:
- moved C407 102.1 mm to (148.6, 130.2)
- moved J102 97.6 mm to (180.0, 151.3), turned to 0 degrees
- moved C601 37.9 mm to (217.7, 130.3), turned to 90 degrees
Connections:
- R413 pad 2: Net-(U401-IO5) -> Net-(U401-IO35)
- U401 pad 17: /T1CK -> /RX2
- U401 pad 18: /T2CK -> /TX2
- U401 pad 29: Net-(U401-IO5) -> /T2CK
- U401 pad 37: /IO8 -> /T1CK
- U401 pad 6: /RX2 -> /IO8
- U401 pad 7: /TX2 -> Net-(U401-IO35)
Routing:
- net GND: track 261.7 -> 588.0 mm, vias 0 -> 6
- net +5VD: track 91.8 -> 369.9 mm, vias 9 -> 16
- net +3.3V: track 85.9 -> 269.8 mm, vias 7 -> 13
- net /SCL-5V: track 31.7 -> 158.6 mm, vias 2 -> 8
- net /SDA-5V: track 40.7 -> 167.1 mm, vias 3 -> 9
- net /D7: track 0.00 -> 87.5 mm, vias 0 -> 2
- net /D0: track 0.00 -> 83.5 mm, vias 0 -> 2
- net /D5: track 0.00 -> 80.6 mm, vias 0 -> 2
- net /D1: track 0.00 -> 80.2 mm, vias 0 -> 2
- net /D6: track 0.00 -> 79.7 mm, vias 0 -> 2
- net /D4: track 0.00 -> 78.2 mm, vias 0 -> 1
- net /D3: track 0.00 -> 76.1 mm, vias 0 -> 2
- net /D2: track 0.00 -> 74.1 mm, vias 0 -> 2
- net Net-(U401-IO4): track 0.00 -> 71.3 mm, vias 0 -> 2
- net Net-(U401-IO2): track 0.00 -> 66.2 mm, vias 0 -> 2
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- added copper zone on B.Cu, net GND
- added copper zone on F.Cu, net GND

Commit message: PCB to control
Parts:
- J102: footprint Connector_Harwin:Harwin_M20-89004xx_1x04_P2.54mm_Horizontal -> Connector_JST:JST_GH_SM04B-GHS-TB_1x04-1MP_P1.25mm_Horizontal
- U205: value MCP23017_SO -> MCP23017_SS; footprint Package_SO:SOIC-28W_7.5x17.9mm_P1.27mm -> Package_SO:SSOP-28_5.3x10.2mm_P0.65mm
- moved R212 6.95 mm to (142.7, 90.8), turned to 90 degrees
- moved R210 5.21 mm to (141.1, 90.8), turned to 90 degrees
- moved U205 4.27 mm to (149.6, 97.0)
- moved R207 4.01 mm to (139.4, 90.8), turned to 90 degrees
- moved J101 0.27 mm to (139.6, 148.3)
- moved J102 0.13 mm to (180.0, 151.1)
Connections:
- C401 pad 1: /ESP32 Module/RESET -> /RESET
- D401 pad 2: +3V3 -> +3.3V
- D402 pad 2: +3V3 -> +3.3V
- R401 pad 1: /ESP32 Module/RESET -> /RESET
- R404 pad 2: /ESP32 Module/RESET -> /RESET
- SW102 pad 2: /ESP32 Module/RESET -> /RESET
- U205 pad 18: /I2C_Peripherique/RESET -> /RESET
- U401 pad 3: /ESP32 Module/RESET -> /RESET
Routing:
- net /RESET: track 0.00 -> 189.1 mm, vias 0 -> 6
- net +3.3V: track 269.8 -> 383.1 mm, vias 13 -> 14
- net /ESP32 Module/RESET: track 82.9 -> 0.00 mm, vias 3 -> 0
- net /RW: track 0.00 -> 72.3 mm, vias 0 -> 2
- net GND: track 588.0 -> 657.6 mm, vias 6 -> 29
- net Net-(U401-IO35): track 0.00 -> 67.7 mm, vias 0 -> 2
- net /SCK: track 0.00 -> 66.1 mm, vias 0 -> 1
- net /SCS: track 0.00 -> 65.2 mm, vias 0 -> 1
- net /E: track 0.00 -> 61.7 mm, vias 0 -> 3
- net +5VD: track 369.9 -> 430.1 mm, vias 16 -> 18
- net /SDO: track 0.00 -> 56.9 mm, vias 0 -> 1
- net /SDI: track 0.00 -> 54.7 mm, vias 0 -> 1
- net /RS: track 0.00 -> 49.7 mm, vias 0 -> 1
- net /RX1: track 0.00 -> 36.2 mm, vias 0 -> 2
- net /TX1: track 0.00 -> 32.8 mm
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