File: KICAD/CPU_ESP/V0.1/CPU/CPU.kicad_pcb (KiCad board)
At the start: 2 copper layers, 100 x 100 mm, 82 parts, among them J101 USB_B_Mini, J102 Conn_01x04, J501 Conn_02x20_Odd_Even, J502 Conn_02x20_Odd_Even, Q601 BSR19, Q602 BSR19, SW101 SW_Push_45deg, SW102 SW_Push_45deg, U201 LM75A, U202 PCA9306, U203 PCF8563T, U204 TCA9544A, U205 MCP23017_SS, U207 AT24CS01-SSHM, U301 LM1117DT-2.5, U401 ESP32-WROOM-32, U402 FT232RL, U403 TJA1051T, U601 SAA1064T, Y201 32.278kHz

Commit message: PCB Update
Parts:
- U203: footprint Package_SO:SOIC-8_3.9x4.9mm_P1.27mm -> Package_SO:MSOP-8_3x3mm_P0.65mm
- moved U203 1.00 mm to (158.0, 114.0)
Routing:
- net GND: track 657.6 -> 673.6 mm
- net /SCL-5V: track 158.2 -> 156.5 mm
