File: KICAD/CPU_ESP/V0.2/CPU/I2C.kicad_sch (KiCad schematic)
At the start: 32 parts, among them U201 LM75A, U202 PCA9306, U203 PCF8563T, U204 TCA9544A, U205 MCP23017_SS, U207 AT24CS01-SSHM, Y201 32.278kHz

Commit message: KICADUpdate
Parts:
- C203: value 10n -> 10p
- D201: footprint Diode_SMD:D_1206_3216Metric -> Diode_SMD:D_2010_5025Metric_Pad1.52x2.65mm_HandSolder
- U201: footprint Package_SO:SOIC-8_3.9x4.9mm_P1.27mm -> Package_SO:MSOP-8_3x3mm_P0.65mm
Changed lines of the file:
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@@
 			)
 		)
-		(property "Value" "10n"
+		(property "Value" "10p"
 			(at 41.91 59.6899 0)
 			(effects
@@
 			)
 		)
-		(property "Footprint" "Diode_SMD:D_1206_3216Metric"
+		(property "Footprint" "Diode_SMD:D_2010_5025Metric_Pad1.52x2.65mm_HandSolder"
 			(at 21.59 29.21 0)
 			(effects
@@
 		)
 		(property "TITLE" ""
+			(at 21.59 29.21 0)
+			(effects
+				(font
+					(size 1.27 1.27)
+				)
+				(hide yes)
+			)
+		)
+		(property "UART" ""
 			(at 21.59 29.21 0)
 			(effects
@@
 			)
 		)
-		(property "Footprint" "Package_SO:SOIC-8_3.9x4.9mm_P1.27mm"
+		(property "Footprint" "Package_SO:MSOP-8_3x3mm_P0.65mm"
 			(at 30.226 105.41 0)
 			(effects
@@
 			(at 33.02 105.41 0)
 			(effects
+				(font
+					(size 1.27 1.27)
+				)
+				(hide yes)
+			)
+		)
+		(property "UART" ""
+			(at 33.02 105.41 0)
+			(effects
