File: KICAD/CPU_ESP/V0.2/CPU/Power.kicad_sch (KiCad schematic)
At the start: 7 parts, among them U301 LM1117DT-2.5

Commit message: KICADUpdate
Parts:
- added C305: 10µ/10V, Capacitor_Tantalum_SMD:CP_EIA-3216-12_Kemet-S_HandSolder, symbol Device:C_Polarized_Small
- C301: value 22µ -> 10µ/10V; footprint Capacitor_Tantalum_SMD:CP_EIA-3216-10_Kemet-I -> Capacitor_Tantalum_SMD:CP_EIA-3216-12_Kemet-S_HandSolder
- C304: value 22µ -> 10µ/10V; footprint Capacitor_Tantalum_SMD:CP_EIA-3528-21_Kemet-B -> Capacitor_Tantalum_SMD:CP_EIA-3216-12_Kemet-S_HandSolder
Connections:
- net +5VD: now also C305.1
- net GND: now also C305.2
Other:
- moved on the sheet: C302
