File: KICAD/CPU_ESP/V0.4/CPU/CPU.kicad_pcb (KiCad board)
At the start: 2 copper layers, 95.2 x 95.2 mm, 90 parts, among them J101 USB_B_Micro, J102 Conn_01x04, J501 Conn_02x20_Odd_Even, J502 Conn_02x20_Odd_Even, Q401 BC817, Q402 BC807, Q601 BSR19, Q602 BSR19, SW101 SW_Push_45deg, SW102 SW_Push_45deg, U201 LM75A, U202 PCA9306, U203 PCF8563T, U204 TCA9544A, U205 MCP23017_SS, U207 AT24CS01-SSHM, U301 LM1117DT-2.5, U401 ESP32-WROOM-32, U402 FT4232H, U403 TJA1051T, U404 93C46, U405 74HC02, U406 74HC244, U601 SAA1064T, Y201 32.278kHz, Y401 12Mhz

Commit message: KICAD update
Parts:
- removed C405, C406: 27P, Capacitor_SMD:C_0603_1608Metric
- removed C407: 10µ/10V, Capacitor_Tantalum_SMD:CP_EIA-3216-12_Kemet-S_HandSolder
- removed R402, R403, R404: 10k, Resistor_SMD:R_0603_1608Metric_Pad0.98x0.95mm_HandSolder
- removed R405: 2K2, Resistor_SMD:R_0603_1608Metric_Pad0.98x0.95mm_HandSolder
- removed R406: 1k, Resistor_SMD:R_0603_1608Metric
- removed R407: 12k, Resistor_SMD:R_0603_1608Metric
- removed U404: 93C46, Package_SO:SOIC-8_5.3x5.3mm_P1.27mm
- removed U405: 74HC02, Package_SO:SOIC-14_3.9x8.7mm_P1.27mm
- removed U406: 74HC244, Package_SO:TSSOP-20_4.4x5mm_P0.5mm
- removed Y401: 12Mhz, Crystal:Crystal_SMD_EuroQuartz_MQ-4Pin_7.0x5.0mm_HandSoldering
- added C306: 10µ/10V, Capacitor_Tantalum_SMD:CP_EIA-3216-12_Kemet-S_HandSolder, F.Cu at (95.0, 146.0)
- added C307: 100n, Capacitor_SMD:C_0603_1608Metric, F.Cu at (96.7, 143.6)
- added FL301: LFCN-80, Filter:Filter_Mini-Circuits_FV1206, F.Cu at (93.5, 141.9)
- C408, C409, L401, L402: moved to F.Cu
- U402: value FT4232H -> XR21V1414-T; footprint Package_QFP:LQFP-64_10x10mm_P0.5mm -> Package_QFP:TQFP-48_7x7mm_P0.5mm
- moved C410 33.0 mm to (100.7, 118.2)
- moved L402 24.7 mm to (91.9, 123.8), turned to -90 degrees
- moved C409 18.7 mm to (93.4, 135.9), turned to -90 degrees
- moved L401 15.8 mm to (97.9, 123.8), turned to -90 degrees
- moved C408 11.2 mm to (102.2, 122.6), turned to 90 degrees
- moved C203 3.97 mm to (105.7, 122.5)
- moved U402 3.77 mm to (104.1, 134.9), turned to 180 degrees
- moved Y201 3.37 mm to (106.5, 116.8), turned to 180 degrees
Connections:
- C408 pad 1: Net-(U402-VPHY) -> Net-(C408-Pad1)
- C409 pad 1: Net-(U402-VPLL) -> Net-(U402-VIO)
- J101 pad 1: /VCCUSB -> /VBUS
- L401 pad 2: Net-(U402-VPHY) -> Net-(C408-Pad1)
- L402 pad 2: Net-(U402-VPLL) -> Net-(U402-VIO)
- U402 pad 10: GND -> unconnected-(U402-GPIOB5/~{RTSB}/RS485B-Pad10)
- U402 pad 11: GND -> unconnected-(U402-GPIOB4/~{CTSB}-Pad11)
- U402 pad 12: Net-(U402-VREGOUT) -> unconnected-(U402-GPIOB3/~{DTRB}-Pad12)
- U402 pad 13: GND -> unconnected-(U402-GPIOB2/~{DSRB}-Pad13)
- U402 pad 14: Net-(U402-~{RESET}) -> unconnected-(U402-GPIOB1/~{CDB}-Pad14)
- U402 pad 15: GND -> unconnected-(U402-GPIOB0/~{RIB}/~{RWKB}-Pad15)
- U402 pad 16: /ESP32 Module/TX0A -> /ESP32 Module/DTR
- U402 pad 17: /ESP32 Module/RX0A -> /ESP32 Module/DSR
- U402 pad 18: /ESP32 Module/RTS -> Net-(C408-Pad1)
- U402 pad 19: /ESP32 Module/CTS -> GND
- U402 pad 2: Net-(U402-OSCI) -> unconnected-(U402-LOW_POWER-Pad2)
- U402 pad 20: +3.3V -> /ESP32 Module/DCD
- U402 pad 21: /ESP32 Module/DTR -> /ESP32 Module/RING
- U402 pad 22: /ESP32 Module/DSR -> /TX2
- U402 pad 23: /ESP32 Module/DCD -> /RX2
- U402 pad 24: /ESP32 Module/RING -> unconnected-(U402-GPIOC5/~{RTSC}/RS485C-Pad24)
- U402 pad 25: GND -> unconnected-(U402-GPIOC4/~{CTSC}-Pad25)
- U402 pad 26: /ESP32 Module/TX1A -> unconnected-(U402-GPIOC3/~{DTRC}-Pad26)
- U402 pad 27: /ESP32 Module/RX1A -> unconnected-(U402-GPIOC2/~{DSRC}-Pad27)
- U402 pad 3: Net-(U402-OSCO) -> unconnected-(U402-GPIOD2/~{DSRD}-Pad3)
- U402 pad 30: unconnected-(U402-BDBUS4-Pad30) -> /ESP32 Module/TX0
- U402 pad 31: +3.3V -> /ESP32 Module/RX0
- U402 pad 32: unconnected-(U402-BDBUS5-Pad32) -> GND
- U402 pad 33: unconnected-(U402-BDBUS6-Pad33) -> Net-(U402-VIO)
- U402 pad 35: GND -> unconnected-(U402-SDA-Pad35)
- U402 pad 36: Net-(U402-~{SUSPEND}) -> unconnected-(U402-SCL-Pad36)
- U402 pad 37: Net-(U402-VREGOUT) -> unconnected-(U402-GPIOD0/~{RID}/~{RWKD}-Pad37)
- U402 pad 38: /ESP32 Module/TX2A -> /TX3
- U402 pad 39: /ESP32 Module/RX2A -> /RX3
- U402 pad 4: Net-(U402-VPHY) -> GND
- U402 pad 40: unconnected-(U402-CDBUS2-Pad40) -> GND
- U402 pad 41: unconnected-(U402-CDBUS3-Pad41) -> GND
- U402 pad 42: +3.3V -> /ESP32 Module/D-
- U402 pad 43: unconnected-(U402-CDBUS4-Pad43) -> /ESP32 Module/D+
- U402 pad 44: unconnected-(U402-CDBUS5-Pad44) -> Net-(U402-VIO)
- U402 pad 45: unconnected-(U402-CDBUS6-Pad45) -> Net-(U402-VIO)
- U402 pad 47: GND -> unconnected-(U402-GPIOD4/~{CTSD}-Pad47)
- U402 pad 48: /ESP32 Module/TX3A -> unconnected-(U402-GPIOD3/~{DTRD}-Pad48)
- U402 pad 5: GND -> Net-(C408-Pad1)
- U402 pad 6: Net-(U402-REF) -> /ESP32 Module/RTS
- U402 pad 7: /ESP32 Module/D- -> /ESP32 Module/CTS
- U402 pad 8: /ESP32 Module/D+ -> /TX1
- U402 pad 9: Net-(U402-VPLL) -> /RX1
Routing:
- net +3.3V: track 420.7 -> 327.2 mm, vias 26 -> 28
- net /ESP32 Module/TX0: track 69.9 -> 122.6 mm, vias 2 -> 4
- net /ESP32 Module/RX3A: track 49.2 -> 0.00 mm, vias 2 -> 0
- net Net-(U402-~{PWREN}): track 44.1 -> 0.00 mm, vias 4 -> 0
- net Net-(U406-2OE): track 36.6 -> 0.00 mm, vias 3 -> 0
- net GND: track 737.7 -> 771.9 mm, vias 18 -> 16
- net Net-(U402-VREGOUT): track 33.5 -> 0.00 mm, vias 2 -> 0
- net /ESP32 Module/RX0A: track 32.1 -> 0.00 mm, vias 4 -> 0
- net Net-(U402-VIO): track 0.00 -> 32.1 mm, vias 0 -> 2
- net /TX3: track 72.9 -> 103.0 mm, vias 1 -> 3
- net /ESP32 Module/RX2A: track 30.0 -> 0.00 mm, vias 2 -> 0
- net /ESP32 Module/TX0A: track 27.9 -> 0.00 mm, vias 2 -> 0
- net /ESP32 Module/TX3A: track 24.5 -> 0.00 mm, vias 2 -> 0
- net /ESP32 Module/RX1A: track 24.3 -> 0.00 mm, vias 2 -> 0
- net Net-(C408-Pad1): track 0.00 -> 22.9 mm
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- added copper zone on B.Cu, net +3.3V
- added copper zone on F.Cu, net +3.3V
Other:
- board text added: "V0.4 CMOS ESP32 DEC-2025"
- board text removed: "V0.3 CMOS ESP32 NOV-2025"
