File: KICAD/CPU_ESP/V0.4/CPU/CPU.kicad_sch (KiCad schematic)
At the start: 4 parts, among them J101 USB_B_Micro, J102 Conn_01x04, SW101 SW_Push_45deg, SW102 SW_Push_45deg

Commit message: KICAD update
Connections:
- net ESP32 Module/VCCUSB renamed VBUS
Other:
- sheet ESP32 Module ports: added none; removed VCCUSB
- sheet Power ports: added VBUSUSB; removed none
Changed lines of the file:
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@@
-	(wire
-		(pts
-			(xy 182.88 121.92) (xy 201.93 121.92)
-		)
-		(stroke
-			(width 0)
-			(type default)
-		)
-	)
 	(wire
 		(pts
@@
 	(wire
 		(pts
+			(xy 92.71 46.99) (xy 95.25 46.99)
+		)
+		(stroke
+			(width 0)
+			(type default)
+		)
+	)
+	(wire
+		(pts
 			(xy 128.27 104.14) (xy 154.94 104.14)
 		)
@@
 		(pts
 			(xy 148.59 149.86) (xy 154.94 149.86)
+		)
+		(stroke
+			(width 0)
+			(type default)
+		)
+	)
+	(wire
+		(pts
+			(xy 199.39 121.92) (xy 201.93 121.92)
 		)
 		(stroke
@@
 		)
 	)
+	(label "VBUS"
+		(at 200.66 121.92 180)
+		(effects
+			(font
+				(size 1.27 1.27)
+			)
+			(justify right bottom)
+		)
+	)
 	(label "D2"
 		(at 191.77 54.61 180)
@@
 			)
 			(justify right bottom)
+		)
+	)
+	(label "VBUS"
+		(at 95.25 46.99 0)
+		(effects
+			(font
+				(size 1.27 1.27)
+			)
+			(justify left bottom)
 		)
 	)
@@
 			)
 		)
-		(pin "VCCUSB" input
-			(at 182.88 121.92 0)
-			(effects
-				(font
-					(size 1.27 1.27)
-				)
-				(justify right)
-			)
-		)
 		(pin "CANH" input
 			(at 182.88 135.89 0)
@@
 			)
 		)
+		(pin "VBUSUSB" input
+			(at 92.71 46.99 0)
+			(effects
+				(font
+					(size 1.27 1.27)
+				)
+				(justify right)
+			)
+		)
