File: KICAD/CPU_ESP/V0.4/CPU/ESP32.kicad_sch (KiCad schematic)
At the start: 24 parts, among them Q401 BC817, Q402 BC807, U401 ESP32-WROOM-32, U402 XR21V1414-T, U403 TJA1051T

Commit message: KICAD update
Connections:
- net GND: now also U402.1 (GND)
- net at C409.1, L402.2, U402.33 (VCC)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: now also U402.44 (VCC), U402.45 (VCC); no longer U402.5 (VCC)
- net at C408.1, L401.2, U402.18 (VCC): now also U402.5 (VCC); no longer U402.44 (VCC), U402.45 (VCC)
