File: KICAD/CPU_ESP/V0.4/CPU/Power.kicad_sch (KiCad schematic)
At the start: 8 parts, among them U301 LM1117DT-2.5

Commit message: KICAD update
Parts:
- added C306: 10µ/10V, Capacitor_Tantalum_SMD:CP_EIA-3216-12_Kemet-S_HandSolder, symbol Device:C_Polarized_Small
- added C307: 100n, Capacitor_SMD:C_0603_1608Metric, symbol Device:C_Small
- added FL301: LFCN-80, Filter:Filter_Mini-Circuits_FV1206, symbol RF_Filter:LFCN-80
Connections:
- net +5VD: now also FL301.3 (OUT)
- net GND: now also C306.2, C307.2, FL301.2 (GND), FL301.4 (GND)
- new net VBUSUSB: C306.1, C307.1, FL301.1 (IN)
